File: kicad/kicad.kicad_pcb (KiCad board)
At the start: 2 copper layers, 231 parts, among them sw1 Esc, sw10 Z, sw100 Num5, sw101 Num6, sw102 Num2, sw103 Num1, sw104 Num0, sw105 mPlay, sw106 mFwd, sw107 Num/, sw108 Num*, sw109 Num8, sw11 LCtrl, sw110 Num9, sw111 Num-, sw112 Num+, sw113 NumEnter, sw114 Num3, sw115 Num., sw12 LSys, sw13 F2, sw14 F3, sw15 2, sw16 3, sw17 W, sw18 E, sw19 S, sw2 F1, sw20 D, sw21 X, sw22 C, sw23 LAlt, sw24 THome, sw25 F4, sw26 F5, sw27 4, sw28 5, sw29 R, sw3 Tilda, sw30 T, sw31 F, sw32 G, sw33 V, sw34 B, sw35 LSpace, sw36 TLeft, sw37 F6, sw38 F7, sw39 6, sw4 1, sw40 7, sw41 Y, sw42 U, sw43 H, sw44 J, sw45 N, sw46 M, sw47 TUp, sw48 TDown, sw49 F8, sw5 Tab, sw50 F9, sw51 8, sw52 9, sw53 I, sw54 O, sw55 K, sw56 L, sw57 ,, sw58 ., sw59 RSpace, sw6 Q, sw60 TRight, sw61 F10, sw62 F11, sw63 0, sw64 -, sw65 P, sw66 [, sw67 ;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

Commit message: startup pcb
Parts:
- D1, D10, D100, D101, D102, D103, D104, D105, D106, D107, D108, D109, D11, D110, D111, D112, D113, D114, D115, D12, D13, D14, D15, D16, D17, D18, D19, D2, D20, D21, D22, D23, D24, D25, D26, D27, D28, D29, D3, D30, D31, D32, D33, D34, D35, D36, D37, D38, D39, D4, D40, D41, D42, D43, D44, D45, D46, D47, D48, D49, D5, D50, D51, D52, D53, D54, D55, D56, D57, D58, D59, D6, D60, D61, D62, D63, D64, D65, D66, D67, D68, D69, D7, D70, D71, D72, D73, D74, D75, D76, D77, D78, D79, D8, D80, D81, D82, D83, D84, D85, D86, D87, D88, D89, D9, D90, D91, D92, D93, D94, D95, D96, D97, D98, D99: moved to B.Cu
- sw100: value Num5 -> N5
- sw101: value Num6 -> N6
- sw102: value Num2 -> N2
- sw103: value Num1 -> N1
- sw104: value Num0 -> N0
- sw105: value mPlay -> MPlay
- sw106: value mFwd -> MFwd
- sw107: value Num/ -> NSlash
- sw108: value Num* -> NStar
- sw109: value Num8 -> N8
- sw110: value Num9 -> N9
- sw111: value Num- -> NMinus
- sw112: value Num+ -> NPlus
- sw113: value NumEnter -> NEnter
- sw114: value Num3 -> N3
- sw115: value Num. -> NPeriod
- sw57: value , -> Comma
- sw58: value . -> Period
- sw64: value - -> Minus
- sw66: value [ -> LBrack
- sw67: value ; -> Semi
- sw68: value ' -> Quote
- sw69: value / -> FSlash
- sw70: footprint Button_Switch_Keyboard:SW_Cherry_MX_2.75u_PCB -> Button_Switch_Keyboard:SW_Cherry_MX_1.00u_PCB
- sw75: value = -> Equals
- sw77: value ] -> RBrack
- sw78: value \ -> BSlash
- sw83: value ScrLck -> Scroll
- sw89: value Num4 -> N4
- sw94: value FN -> Fn
- sw95: value mBack -> MBack
- sw97: value NumLck -> NLock
- sw99: value Num7 -> N7
- moved MCU1 854.2 mm to (269.1, -161.9)
- moved D106 741.0 mm to (342.8, -128.6)
- moved D107 735.0 mm to (304.7, -109.5)
- moved D100 729.3 mm to (304.7, -71.4)
- moved D94 722.3 mm to (285.7, -128.6)
- moved D102 719.4 mm to (304.7, -52.4)
- moved D95 717.2 mm to (304.7, -128.6)
- moved D113 702.9 mm to (342.8, -42.9)
- moved D108 689.8 mm to (323.8, -109.5)
- moved D104 671.8 mm to (295.2, -33.3)
- moved D110 658.2 mm to (323.8, -90.5)
- moved D99 657.4 mm to (285.7, -90.5)
- moved D115 657.1 mm to (323.8, -33.3)
- moved D111 652.6 mm to (342.8, -109.5)
- moved D76 635.7 mm to (200.0, -109.5)
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
Commit message: route rows
Parts:
- moved sw1 159.0 mm to (0.00, 9.53)
- moved sw10 159.0 mm to (42.9, 85.7)
- moved sw100 159.0 mm to (361.9, 66.7)
- moved sw101 159.0 mm to (381.0, 66.7)
- moved sw102 159.0 mm to (361.9, 85.7)
- moved sw103 159.0 mm to (342.9, 85.7)
- moved sw104 159.0 mm to (352.4, 104.8)
- moved sw105 159.0 mm to (381.0, 9.53)
- moved sw106 159.0 mm to (400.1, 9.53)
- moved sw107 159.0 mm to (361.9, 28.6)
- moved sw108 159.0 mm to (381.0, 28.6)
- moved sw109 159.0 mm to (361.9, 47.6)
- moved sw11 159.0 mm to (2.38, 104.8)
- moved sw110 159.0 mm to (381.0, 47.6)
- moved sw111 159.0 mm to (400.1, 28.6)
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Routing:
- net Net-(sw110-Pad1): track 0.00 -> 517.0 mm
- net Net-(sw108-Pad1): track 0.00 -> 510.6 mm
- net Net-(sw115-Pad1): track 0.00 -> 509.3 mm
- net Net-(sw10-Pad1): track 0.00 -> 497.7 mm
- net Net-(sw100-Pad1): track 0.00 -> 491.9 mm
- net Net-(sw101-Pad1): track 0.00 -> 491.6 mm
- net Net-(sw106-Pad1): track 0.00 -> 489.8 mm
- net Net-(sw1-Pad1): track 0.00 -> 474.7 mm
- net Net-(sw104-Pad1): track 0.00 -> 473.7 mm
- net Net-(sw109-Pad1): track 0.00 -> 472.3 mm
- net Net-(sw102-Pad1): track 0.00 -> 471.3 mm
- net Net-(sw107-Pad1): track 0.00 -> 471.0 mm
- net Net-(D75-Pad1): track 0.00 -> 9.14 mm
- net Net-(D85-Pad1): track 0.00 -> 8.67 mm
- net Net-(D108-Pad1): track 0.00 -> 8.67 mm
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
Commit message: route columns
Parts:
- added U1: AMS1117-3.3, Package_TO_SOT_SMD:SOT-223-3_TabPin2, F.Cu at (287.5, -175.0)
Connections:
- D1 pad 2: Net-(D1-Pad2) -> COLUMN8
- D10 pad 2: Net-(D1-Pad2) -> COLUMN8
- D105 pad 2: Net-(D105-Pad2) -> COLUMN1
- D106 pad 2: Net-(D105-Pad2) -> COLUMN1
- D107 pad 2: Net-(D105-Pad2) -> COLUMN1
- D108 pad 2: Net-(D105-Pad2) -> COLUMN1
- D109 pad 2: Net-(D105-Pad2) -> COLUMN1
- D11 pad 2: Net-(D1-Pad2) -> COLUMN8
- D110 pad 2: Net-(D105-Pad2) -> COLUMN1
- D111 pad 2: Net-(D105-Pad2) -> COLUMN1
- D112 pad 2: Net-(D105-Pad2) -> COLUMN1
- D113 pad 2: Net-(D105-Pad2) -> COLUMN1
- D114 pad 2: Net-(D105-Pad2) -> COLUMN1
- D115 pad 2: Net-(D105-Pad2) -> COLUMN1
- D12 pad 2: unconnected-(D12-Pad2) -> COLUMN8
- D2 pad 2: Net-(D1-Pad2) -> COLUMN8
- D25 pad 2: Net-(D25-Pad2) -> COLUMN7
- D26 pad 2: Net-(D25-Pad2) -> COLUMN7
- D27 pad 2: Net-(D25-Pad2) -> COLUMN7
- D28 pad 2: Net-(D25-Pad2) -> COLUMN7
- D29 pad 2: Net-(D25-Pad2) -> COLUMN7
- D3 pad 2: Net-(D1-Pad2) -> COLUMN8
- D30 pad 2: Net-(D25-Pad2) -> COLUMN7
- D31 pad 2: Net-(D25-Pad2) -> COLUMN7
- D32 pad 2: Net-(D25-Pad2) -> COLUMN7
- D33 pad 2: Net-(D25-Pad2) -> COLUMN7
- D34 pad 2: Net-(D25-Pad2) -> COLUMN7
- D35 pad 2: Net-(D25-Pad2) -> COLUMN7
- D36 pad 2: Net-(D25-Pad2) -> COLUMN7
- D37 pad 2: Net-(D37-Pad2) -> COLUMN6
- D38 pad 2: Net-(D37-Pad2) -> COLUMN6
- D39 pad 2: Net-(D37-Pad2) -> COLUMN6
- D4 pad 2: Net-(D1-Pad2) -> COLUMN8
- D40 pad 2: Net-(D37-Pad2) -> COLUMN6
- D41 pad 2: Net-(D37-Pad2) -> COLUMN6
- D42 pad 2: Net-(D37-Pad2) -> COLUMN6
- D43 pad 2: Net-(D37-Pad2) -> COLUMN6
- D44 pad 2: Net-(D37-Pad2) -> COLUMN6
- D45 pad 2: Net-(D37-Pad2) -> COLUMN6
- D46 pad 2: Net-(D37-Pad2) -> COLUMN6
- D47 pad 2: Net-(D37-Pad2) -> COLUMN6
- D48 pad 2: Net-(D37-Pad2) -> COLUMN6
- D49 pad 2: Net-(D49-Pad2) -> COLUMN5
- D5 pad 2: Net-(D1-Pad2) -> COLUMN8
- D50 pad 2: Net-(D49-Pad2) -> COLUMN5
- D51 pad 2: Net-(D49-Pad2) -> COLUMN5
- D52 pad 2: Net-(D49-Pad2) -> COLUMN5
- D53 pad 2: Net-(D49-Pad2) -> COLUMN5
- D54 pad 2: Net-(D49-Pad2) -> COLUMN5
- D55 pad 2: Net-(D49-Pad2) -> COLUMN5
- D56 pad 2: Net-(D49-Pad2) -> COLUMN5
- D57 pad 2: Net-(D49-Pad2) -> COLUMN5
- D58 pad 2: Net-(D49-Pad2) -> COLUMN5
- D59 pad 2: Net-(D49-Pad2) -> COLUMN5
- D6 pad 2: Net-(D1-Pad2) -> COLUMN8
- D60 pad 2: Net-(D49-Pad2) -> COLUMN5
- D61 pad 2: Net-(D61-Pad2) -> COLUMN4
- D62 pad 2: Net-(D61-Pad2) -> COLUMN4
- D63 pad 2: Net-(D61-Pad2) -> COLUMN4
- D64 pad 2: Net-(D61-Pad2) -> COLUMN4
- D65 pad 2: Net-(D61-Pad2) -> COLUMN4
- D66 pad 2: Net-(D61-Pad2) -> COLUMN4
- D67 pad 2: Net-(D61-Pad2) -> COLUMN4
- D68 pad 2: Net-(D61-Pad2) -> COLUMN4
- D69 pad 2: Net-(D61-Pad2) -> COLUMN4
- D7 pad 2: Net-(D1-Pad2) -> COLUMN8
- D70 pad 2: Net-(D61-Pad2) -> COLUMN4
- D71 pad 2: Net-(D61-Pad2) -> COLUMN4
- D72 pad 2: Net-(D61-Pad2) -> COLUMN4
- D73 pad 2: Net-(D73-Pad2) -> COLUMN3
- D74 pad 2: Net-(D73-Pad2) -> COLUMN3
- D75 pad 2: Net-(D73-Pad2) -> COLUMN3
- D76 pad 2: Net-(D73-Pad2) -> COLUMN3
- D77 pad 2: Net-(D73-Pad2) -> COLUMN3
- D78 pad 2: Net-(D73-Pad2) -> COLUMN3
- D79 pad 2: Net-(D73-Pad2) -> COLUMN3
- D8 pad 2: Net-(D1-Pad2) -> COLUMN8
- D80 pad 2: Net-(D73-Pad2) -> COLUMN3
- D81 pad 2: Net-(D73-Pad2) -> COLUMN3
- D82 pad 2: Net-(D73-Pad2) -> COLUMN3
- D83 pad 2: Net-(D83-Pad2) -> COLUMN2
- D84 pad 2: Net-(D83-Pad2) -> COLUMN2
- D85 pad 2: Net-(D83-Pad2) -> COLUMN2
- D86 pad 2: Net-(D83-Pad2) -> COLUMN2
- D87 pad 2: Net-(D83-Pad2) -> COLUMN2
- D88 pad 2: Net-(D83-Pad2) -> COLUMN2
- D89 pad 2: Net-(D83-Pad2) -> COLUMN2
- D9 pad 2: Net-(D1-Pad2) -> COLUMN8
- D90 pad 2: unconnected-(D90-Pad2) -> COLUMN2
- D91 pad 2: Net-(D83-Pad2) -> COLUMN2
- D92 pad 2: Net-(D83-Pad2) -> COLUMN2
- D93 pad 2: Net-(D83-Pad2) -> COLUMN2
- MCU1 pad 13: unconnected-(MCU1-Pad13) -> +3.3V
- MCU1 pad 16: unconnected-(MCU1-Pad16) -> COLUMN8
- MCU1 pad 17: unconnected-(MCU1-Pad17) -> COLUMN7
- MCU1 pad 20: unconnected-(MCU1-Pad20) -> COLUMN6
- MCU1 pad 21: unconnected-(MCU1-Pad21) -> COLUMN5
- MCU1 pad 22: unconnected-(MCU1-Pad22) -> COLUMN4
- MCU1 pad 23: unconnected-(MCU1-Pad23) -> COLUMN3
- MCU1 pad 24: unconnected-(MCU1-Pad24) -> COLUMN2
- MCU1 pad 25: unconnected-(MCU1-Pad25) -> COLUMN1
- MCU1 pad 26: unconnected-(MCU1-Pad26) -> CAPS_LOCK_LED
- MCU1 pad 27: unconnected-(MCU1-Pad27) -> ROW12
- MCU1 pad 28: unconnected-(MCU1-Pad28) -> ROW11
- MCU1 pad 29: unconnected-(MCU1-Pad29) -> ROW10
- MCU1 pad 30: unconnected-(MCU1-Pad30) -> ROW9
- MCU1 pad 33: unconnected-(MCU1-Pad33) -> ROW8
- MCU1 pad 34: unconnected-(MCU1-Pad34) -> ROW7
- MCU1 pad 35: unconnected-(MCU1-Pad35) -> ROW6
- MCU1 pad 36: unconnected-(MCU1-Pad36) -> ROW5
- MCU1 pad 37: unconnected-(MCU1-Pad37) -> ROW4
- MCU1 pad 38: unconnected-(MCU1-Pad38) -> ROW3
- MCU1 pad 39: unconnected-(MCU1-Pad39) -> ROW2
- MCU1 pad 40: unconnected-(MCU1-Pad40) -> ROW1
- MCU1 pad 44: unconnected-(MCU1-Pad44) -> /USB_DM
- MCU1 pad 45: unconnected-(MCU1-Pad45) -> /USB_DP
- MCU1 pad 46: unconnected-(MCU1-Pad46) -> /SWDIO
- MCU1 pad 49: unconnected-(MCU1-Pad49) -> /SWCLK
- MCU1 pad 60: unconnected-(MCU1-Pad60) -> /BOOT0
- MCU1 pad 7: unconnected-(MCU1-Pad7) -> /NRST
- sw1 pad 1: Net-(sw1-Pad1) -> ROW1
- sw10 pad 1: Net-(sw10-Pad1) -> ROW10
- sw100 pad 1: Net-(sw100-Pad1) -> ROW7
- sw101 pad 1: Net-(sw101-Pad1) -> ROW8
- sw102 pad 1: Net-(sw102-Pad1) -> ROW9
- sw103 pad 1: Net-(sw10-Pad1) -> ROW10
- sw104 pad 1: Net-(sw104-Pad1) -> ROW11
- sw105 pad 1: Net-(sw1-Pad1) -> ROW1
- sw106 pad 1: Net-(sw106-Pad1) -> ROW2
- sw107 pad 1: Net-(sw107-Pad1) -> ROW3
- sw108 pad 1: Net-(sw108-Pad1) -> ROW4
- sw109 pad 1: Net-(sw109-Pad1) -> ROW5
- sw11 pad 1: Net-(sw104-Pad1) -> ROW11
- sw110 pad 1: Net-(sw110-Pad1) -> ROW6
- sw111 pad 1: Net-(sw100-Pad1) -> ROW7
- sw112 pad 1: Net-(sw101-Pad1) -> ROW8
- sw113 pad 1: Net-(sw102-Pad1) -> ROW9
- sw114 pad 1: Net-(sw10-Pad1) -> ROW10
- sw115 pad 1: Net-(sw115-Pad1) -> ROW12
- sw12 pad 1: Net-(sw115-Pad1) -> ROW12
- sw13 pad 1: Net-(sw1-Pad1) -> ROW1
- sw14 pad 1: Net-(sw106-Pad1) -> ROW2
- sw15 pad 1: Net-(sw107-Pad1) -> ROW3
- sw16 pad 1: Net-(sw108-Pad1) -> ROW4
- sw17 pad 1: Net-(sw109-Pad1) -> ROW5
- sw18 pad 1: Net-(sw110-Pad1) -> ROW6
- sw19 pad 1: Net-(sw100-Pad1) -> ROW7
- sw2 pad 1: Net-(sw106-Pad1) -> ROW2
- sw20 pad 1: Net-(sw101-Pad1) -> ROW8
- sw21 pad 1: Net-(sw102-Pad1) -> ROW9
- sw22 pad 1: Net-(sw10-Pad1) -> ROW10
- sw23 pad 1: Net-(sw104-Pad1) -> ROW11
- sw24 pad 1: Net-(sw115-Pad1) -> ROW12
- sw25 pad 1: Net-(sw1-Pad1) -> ROW1
- sw26 pad 1: Net-(sw106-Pad1) -> ROW2
- sw27 pad 1: Net-(sw107-Pad1) -> ROW3
- sw28 pad 1: Net-(sw108-Pad1) -> ROW4
- sw29 pad 1: Net-(sw109-Pad1) -> ROW5
- sw3 pad 1: Net-(sw107-Pad1) -> ROW3
- sw30 pad 1: Net-(sw110-Pad1) -> ROW6
- sw31 pad 1: Net-(sw100-Pad1) -> ROW7
- sw32 pad 1: Net-(sw101-Pad1) -> ROW8
- sw33 pad 1: Net-(sw102-Pad1) -> ROW9
- sw34 pad 1: Net-(sw10-Pad1) -> ROW10
- sw35 pad 1: Net-(sw104-Pad1) -> ROW11
- sw36 pad 1: Net-(sw115-Pad1) -> ROW12
- sw37 pad 1: Net-(sw1-Pad1) -> ROW1
- sw38 pad 1: Net-(sw106-Pad1) -> ROW2
- sw39 pad 1: Net-(sw107-Pad1) -> ROW3
- sw4 pad 1: Net-(sw108-Pad1) -> ROW4
- sw40 pad 1: Net-(sw108-Pad1) -> ROW4
- sw41 pad 1: Net-(sw109-Pad1) -> ROW5
- sw42 pad 1: Net-(sw110-Pad1) -> ROW6
- sw43 pad 1: Net-(sw100-Pad1) -> ROW7
- sw44 pad 1: Net-(sw101-Pad1) -> ROW8
- sw45 pad 1: Net-(sw102-Pad1) -> ROW9
- sw46 pad 1: Net-(sw10-Pad1) -> ROW10
- sw47 pad 1: Net-(sw104-Pad1) -> ROW11
- sw48 pad 1: Net-(sw115-Pad1) -> ROW12
- sw49 pad 1: Net-(sw1-Pad1) -> ROW1
- sw5 pad 1: Net-(sw109-Pad1) -> ROW5
- sw50 pad 1: Net-(sw106-Pad1) -> ROW2
- sw51 pad 1: Net-(sw107-Pad1) -> ROW3
- sw52 pad 1: Net-(sw108-Pad1) -> ROW4
- sw53 pad 1: Net-(sw109-Pad1) -> ROW5
- sw54 pad 1: Net-(sw110-Pad1) -> ROW6
- sw55 pad 1: Net-(sw100-Pad1) -> ROW7
- sw56 pad 1: Net-(sw101-Pad1) -> ROW8
- sw57 pad 1: Net-(sw102-Pad1) -> ROW9
- sw58 pad 1: Net-(sw10-Pad1) -> ROW10
- sw59 pad 1: Net-(sw104-Pad1) -> ROW11
- sw6 pad 1: Net-(sw110-Pad1) -> ROW6
- sw60 pad 1: Net-(sw115-Pad1) -> ROW12
- sw61 pad 1: Net-(sw1-Pad1) -> ROW1
- sw62 pad 1: Net-(sw106-Pad1) -> ROW2
- sw63 pad 1: Net-(sw107-Pad1) -> ROW3
- sw64 pad 1: Net-(sw108-Pad1) -> ROW4
- sw65 pad 1: Net-(sw109-Pad1) -> ROW5
- sw66 pad 1: Net-(sw110-Pad1) -> ROW6
- sw67 pad 1: Net-(sw100-Pad1) -> ROW7
- sw68 pad 1: Net-(sw101-Pad1) -> ROW8
- sw69 pad 1: Net-(sw102-Pad1) -> ROW9
- sw7 pad 1: Net-(sw100-Pad1) -> ROW7
- sw70 pad 1: Net-(sw10-Pad1) -> ROW10
- sw71 pad 1: Net-(sw104-Pad1) -> ROW11
- sw72 pad 1: Net-(sw115-Pad1) -> ROW12
- sw73 pad 1: Net-(sw1-Pad1) -> ROW1
- sw74 pad 1: Net-(sw106-Pad1) -> ROW2
- sw75 pad 1: Net-(sw107-Pad1) -> ROW3
- sw76 pad 1: Net-(sw108-Pad1) -> ROW4
- sw77 pad 1: Net-(sw109-Pad1) -> ROW5
- sw78 pad 1: Net-(sw110-Pad1) -> ROW6
- sw79 pad 1: Net-(sw100-Pad1) -> ROW7
- sw8 pad 1: Net-(sw101-Pad1) -> ROW8
- sw80 pad 1: Net-(sw10-Pad1) -> ROW10
- sw81 pad 1: Net-(sw104-Pad1) -> ROW11
- sw82 pad 1: Net-(sw115-Pad1) -> ROW12
- sw83 pad 1: Net-(sw1-Pad1) -> ROW1
- sw84 pad 1: Net-(sw106-Pad1) -> ROW2
- sw85 pad 1: Net-(sw107-Pad1) -> ROW3
- sw86 pad 1: Net-(sw108-Pad1) -> ROW4
- sw87 pad 1: Net-(sw109-Pad1) -> ROW5
- sw88 pad 1: Net-(sw110-Pad1) -> ROW6
- sw89 pad 1: Net-(sw101-Pad1) -> ROW8
- sw9 pad 1: Net-(sw102-Pad1) -> ROW9
- sw90 pad 1: Net-(sw102-Pad1) -> ROW9
- sw91 pad 1: Net-(sw10-Pad1) -> ROW10
- sw92 pad 1: Net-(sw104-Pad1) -> ROW11
- sw93 pad 1: Net-(sw115-Pad1) -> ROW12
- sw94 pad 1: Net-(sw1-Pad1) -> ROW1
- sw95 pad 1: Net-(sw106-Pad1) -> ROW2
- sw96 pad 1: Net-(sw107-Pad1) -> ROW3
- sw97 pad 1: Net-(sw108-Pad1) -> ROW4
- sw98 pad 1: Net-(sw109-Pad1) -> ROW5
- sw99 pad 1: Net-(sw110-Pad1) -> ROW6
Routing:
- net ROW6: track 0.00 -> 517.0 mm
- net Net-(sw110-Pad1): track 517.0 -> 0.00 mm
- net ROW4: track 0.00 -> 510.6 mm
- net Net-(sw108-Pad1): track 510.6 -> 0.00 mm
- net ROW12: track 0.00 -> 509.3 mm
- net Net-(sw115-Pad1): track 509.3 -> 0.00 mm
- net ROW10: track 0.00 -> 497.7 mm
- net Net-(sw10-Pad1): track 497.7 -> 0.00 mm
- net ROW7: track 0.00 -> 491.9 mm
- net Net-(sw100-Pad1): track 491.9 -> 0.00 mm
- net ROW8: track 0.00 -> 491.6 mm
- net Net-(sw101-Pad1): track 491.6 -> 0.00 mm
- net ROW2: track 0.00 -> 489.8 mm
- net Net-(sw106-Pad1): track 489.8 -> 0.00 mm
- net ROW1: track 0.00 -> 474.7 mm
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
Commit message: working towards merge
Connections:
- D12 pad 2: COLUMN8 -> unconnected-(D12-Pad2)
- D90 pad 2: COLUMN2 -> unconnected-(D90-Pad2)
Routing:
- net COLUMN8: track 290.1 -> 274.6 mm
- net unconnected-(D12-Pad2): track 0.00 -> 14.1 mm
- net COLUMN2: track 278.2 -> 265.3 mm
- net unconnected-(D90-Pad2): track 0.00 -> 11.8 mm
Changed lines of the file:
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@@
   (net 172 "Net-(D114-Pad1)")
   (net 173 "Net-(D115-Pad1)")
+  (net 174 "unconnected-(D12-Pad2)")
+  (net 175 "unconnected-(D90-Pad2)")
   (footprint "Button_Switch_Keyboard:SW_Cherry_MX_1.00u_PCB" (layer "F.Cu")
     (at 114.3 28.575)
@@
       (net 67 "Net-(D12-Pad1)") (pinfunction "K") (pintype "input"))
     (pad "2" smd rect (at 1.4 0) (size 1.1 1.1) (layers "B.Cu" "B.Paste" "B.Mask")
-      (net 2 "COLUMN8") (pinfunction "A") (pintype "input"))
+      (net 174 "unconnected-(D12-Pad2)") (pinfunction "A") (pintype "input"))
     (model "${KICAD6_3DMODEL_DIR}/Diode_SMD.3dshapes/D_SOD-123F.wrl"
       (offset (xyz 0 0 0))
@@
       (net 147 "Net-(D90-Pad1)") (pinfunction "K") (pintype "input"))
     (pad "2" smd rect (at 1.4 0) (size 1.1 1.1) (layers "B.Cu" "B.Paste" "B.Mask")
-      (net 21 "COLUMN2") (pinfunction "A") (pintype "input"))
+      (net 175 "unconnected-(D90-Pad2)") (pinfunction "A") (pintype "input"))
     (model "${KICAD6_3DMODEL_DIR}/Diode_SMD.3dshapes/D_SOD-123F.wrl"
       (offset (xyz 0 0 0))
@@
   (segment (start 15.84 95.92) (end 17.018 94.742) (width 0.25) (layer "B.Cu") (net 2))
   (segment (start 41.7625 98.1915) (end 41.148 98.806) (width 0.25) (layer "B.Cu") (net 2))
-  (segment (start 24.384 117.348) (end 12.954 117.348) (width 0.25) (layer "B.Cu") (net 2))
   (segment (start 10.8806 95.92) (end 15.84 95.92) (width 0.25) (layer "B.Cu") (net 2))
   (segment (start 10.252 114.97) (end 11.938 113.284) (width 0.25) (layer "B.Cu") (net 2))
-  (segment (start 12.954 117.348) (end 11.938 116.332) (width 0.25) (layer "B.Cu") (net 2))
   (segment (start 17.018 94.742) (end 17.018 93.472) (width 0.25) (layer "B.Cu") (net 2))
   (segment (start 1.281 114.97) (end 10.252 114.97) (width 0.25) (layer "B.Cu") (net 2))
@@
   (segment (start 8.636 43.942) (end 17.018 52.324) (width 0.25) (layer "B.Cu") (net 2))
   (segment (start 16.348 76.87) (end 17.018 76.2) (width 0.25) (layer "B.Cu") (net 2))
-  (segment (start 25.0935 116.6385) (end 24.384 117.348) (width 0.25) (layer "B.Cu") (net 2))
   (segment (start 18.288 59.944) (end 17.018 61.214) (width 0.25) (layer "B.Cu") (net 2))
   (segment (start 24.892 98.806) (end 17.018 90.932) (width 0.25) (layer "B.Cu") (net 2))
@@
   (segment (start 27.432 59.436) (end 26.924 59.944) (width 0.25) (layer "B.Cu") (net 2))
   (segment (start 17.018 76.454) (end 17.018 76.2) (width 0.25) (layer "B.Cu") (net 2))
-  (segment (start 25.0935 114.97) (end 25.0935 116.6385) (width 0.25) (layer "B.Cu") (net 2))
   (segment (start 8.382 22.606) (end 35.814 22.606) (width 0.25) (layer "B.Cu") (net 2))
   (segment (start 7.112 23.876) (end 8.382 22.606) (width 0.25) (layer "B.Cu") (net 2))
@@
   (segment (start 293.624 116.586) (end 294.894 117.856) (width 0.25) (layer "B.Cu") (net 21))
   (segment (start 284.65 38.77) (end 292.516 38.77) (width 0.25) (layer "B.Cu") (net 21))
-  (segment (start 294.132 98.806) (end 293.37 99.568) (width 0.25) (layer "B.Cu") (net 21))
   (segment (start 303.022 117.856) (end 320.548 117.856) (width 0.25) (layer "B.Cu") (net 21))
   (segment (start 293.37 60.96) (end 293.37 80.518) (width 0.25) (layer "B.Cu") (net 21))
@@
   (segment (start 303.7 117.178) (end 303.022 117.856) (width 0.25) (layer "B.Cu") (net 21))
   (segment (start 303.022 23.368) (end 297.688 23.368) (width 0.25) (layer "B.Cu") (net 21))
-  (segment (start 303.7 97.706) (end 302.6 98.806) (width 0.25) (layer "B.Cu") (net 21))
   (segment (start 293.37 60.706) (end 293.37 60.96) (width 0.25) (layer "B.Cu") (net 21))
   (segment (start 294.386 59.69) (end 293.37 60.706) (width 0.25) (layer "B.Cu") (net 21))
@@
   (segment (start 302.514 59.69) (end 294.386 59.69) (width 0.25) (layer "B.Cu") (net 21))
   (segment (start 292.608 59.69) (end 293.37 60.452) (width 0.25) (layer "B.Cu") (net 21))
-  (segment (start 303.7 95.92) (end 303.7 97.706) (width 0.25) (layer "B.Cu") (net 21))
   (segment (start 341.8 76.87) (end 341.8 78.316) (width 0.25) (layer "B.Cu") (net 21))
   (segment (start 293.37 80.01) (end 293.37 80.518) (width 0.25) (layer "B.Cu") (net 21))
@@
   (segment (start 293.37 80.518) (end 293.37 99.568) (width 0.25) (layer "B.Cu") (net 21))
   (segment (start 303.022 40.386) (end 294.132 40.386) (width 0.25) (layer "B.Cu") (net 21))
-  (segment (start 302.6 98.806) (end 294.132 98.806) (width 0.25) (layer "B.Cu") (net 21))
   (segment (start 322.75 21.42) (end 320.802 23.368) (width 0.25) (layer "B.Cu") (net 21))
   (segment (start 294.894 117.856) (end 303.022 117.856) (width 0.25) (layer "B.Cu") (net 21))
@@
   (segment (start 374.65 112.52) (end 374.65 107.315) (width 0.25) (layer "B.Cu") (net 173))
   (segment (start 377.1 114.97) (end 374.65 112.52) (width 0.25) (layer "B.Cu") (net 173))
+  (segment (start 24.384 117.348) (end 12.954 117.348) (width 0.25) (layer "B.Cu") (net 174))
+  (segment (start 25.0935 116.6385) (end 24.384 117.348) (width 0.25) (layer "B.Cu") (net 174))
+  (segment (start 25.0935 114.97) (end 25.0935 116.6385) (width 0.25) (layer "B.Cu") (net 174))
+  (segment (start 303.7 97.706) (end 302.6 98.806) (width 0.25) (layer "B.Cu") (net 175))
+  (segment (start 303.7 95.92) (end 303.7 97.706) (width 0.25) (layer "B.Cu") (net 175))
+  (segment (start 302.6 98.806) (end 294.132 98.806) (width 0.25) (layer "B.Cu") (net 175))
 )
