File: kicad/kicad.kicad_pcb (KiCad board)
At the start: 2 copper layers, 232 parts, among them U1 AMS1117-3.3, sw1 Esc, sw10 Z, sw100 N5, sw101 N6, sw102 N2, sw103 N1, sw104 N0, sw105 MPlay, sw106 MFwd, sw107 NSlash, sw108 NStar, sw109 N8, sw11 LCtrl, sw110 N9, sw111 NMinus, sw112 NPlus, sw113 NEnter, sw114 N3, sw115 NPeriod, sw12 LSys, sw13 F2, sw14 F3, sw15 2, sw16 3, sw17 W, sw18 E, sw19 S, sw2 F1, sw20 D, sw21 X, sw22 C, sw23 LAlt, sw24 THome, sw25 F4, sw26 F5, sw27 4, sw28 5, sw29 R, sw3 Tilda, sw30 T, sw31 F, sw32 G, sw33 V, sw34 B, sw35 LSpace, sw36 TLeft, sw37 F6, sw38 F7, sw39 6, sw4 1, sw40 7, sw41 Y, sw42 U, sw43 H, sw44 J, sw45 N, sw46 M, sw47 TUp, sw48 TDown, sw49 F8, sw5 Tab, sw50 F9, sw51 8, sw52 9, sw53 I, sw54 O, sw55 K, sw56 L, sw57 Comma, sw58 Period, sw59 RSpace, sw6 Q, sw60 TRight, sw61 F10, sw62 F11, sw63 0, sw64 Minus, sw65 P, sw66 LBrack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

Commit message: recover small change lost in merge
Connections:
- D12 pad 2: unconnected-(D12-Pad2) -> COLUMN8
- D90 pad 2: unconnected-(D90-Pad2) -> COLUMN2
Routing:
- net COLUMN8: track 274.6 -> 290.1 mm
- net unconnected-(D12-Pad2): track 14.1 -> 0.00 mm
- net COLUMN2: track 265.3 -> 278.2 mm
- net unconnected-(D90-Pad2): track 11.8 -> 0.00 mm
Changed lines of the file:
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@@
   (net 170 "Net-(D114-Pad1)")
   (net 171 "Net-(D115-Pad1)")
-  (net 172 "unconnected-(D12-Pad2)")
-  (net 173 "unconnected-(D90-Pad2)")
-  (net 174 "/RCC_OSC_IN")
-  (net 175 "/RCC_OSC_OUT")
+  (net 172 "/RCC_OSC_IN")
+  (net 173 "/RCC_OSC_OUT")
   (footprint "Button_Switch_Keyboard:SW_Cherry_MX_1.00u_PCB" (layer "F.Cu")
     (at 114.3 28.575)
@@
       (net 6 "unconnected-(MCU1-Pad4)") (pinfunction "PC15") (pintype "bidirectional"))
     (pad "5" smd roundrect (at -5.675 -1.75) (size 1.55 0.3) (layers "F.Cu" "F.Paste" "F.Mask") (roundrect_rratio 0.25)
-      (net 174 "/RCC_OSC_IN") (pinfunction "PD0") (pintype "input"))
+      (net 172 "/RCC_OSC_IN") (pinfunction "PD0") (pintype "input"))
     (pad "6" smd roundrect (at -5.675 -1.25) (size 1.55 0.3) (layers "F.Cu" "F.Paste" "F.Mask") (roundrect_rratio 0.25)
-      (net 175 "/RCC_OSC_OUT") (pinfunction "PD1") (pintype "input"))
+      (net 173 "/RCC_OSC_OUT") (pinfunction "PD1") (pintype "input"))
     (pad "7" smd roundrect (at -5.675 -0.75) (size 1.55 0.3) (layers "F.Cu" "F.Paste" "F.Mask") (roundrect_rratio 0.25)
       (net 21 "/NRST") (pinfunction "NRST") (pintype "input"))
@@
       (net 65 "Net-(D12-Pad1)") (pinfunction "K") (pintype "input"))
     (pad "2" smd rect (at 1.4 0) (size 1.1 1.1) (layers "B.Cu" "B.Paste" "B.Mask")
-      (net 172 "unconnected-(D12-Pad2)") (pinfunction "A") (pintype "input"))
+      (net 2 "COLUMN8") (pinfunction "A") (pintype "input"))
     (model "${KICAD6_3DMODEL_DIR}/Diode_SMD.3dshapes/D_SOD-123F.wrl"
       (offset (xyz 0 0 0))
@@
       (net 145 "Net-(D90-Pad1)") (pinfunction "K") (pintype "input"))
     (pad "2" smd rect (at 1.4 0) (size 1.1 1.1) (layers "B.Cu" "B.Paste" "B.Mask")
-      (net 173 "unconnected-(D90-Pad2)") (pinfunction "A") (pintype "input"))
+      (net 19 "COLUMN2") (pinfunction "A") (pintype "input"))
     (model "${KICAD6_3DMODEL_DIR}/Diode_SMD.3dshapes/D_SOD-123F.wrl"
       (offset (xyz 0 0 0))
@@
   (segment (start 15.84 95.92) (end 17.018 94.742) (width 0.25) (layer "B.Cu") (net 2))
   (segment (start 41.7625 98.1915) (end 41.148 98.806) (width 0.25) (layer "B.Cu") (net 2))
+  (segment (start 24.384 117.348) (end 12.954 117.348) (width 0.25) (layer "B.Cu") (net 2))
   (segment (start 10.8806 95.92) (end 15.84 95.92) (width 0.25) (layer "B.Cu") (net 2))
   (segment (start 10.252 114.97) (end 11.938 113.284) (width 0.25) (layer "B.Cu") (net 2))
@@
   (segment (start 8.636 43.942) (end 17.018 52.324) (width 0.25) (layer "B.Cu") (net 2))
   (segment (start 16.348 76.87) (end 17.018 76.2) (width 0.25) (layer "B.Cu") (net 2))
+  (segment (start 25.0935 116.6385) (end 24.384 117.348) (width 0.25) (layer "B.Cu") (net 2))
   (segment (start 18.288 59.944) (end 17.018 61.214) (width 0.25) (layer "B.Cu") (net 2))
+  (segment (start 12.954 117.348) (end 11.938 116.332) (width 0.25) (layer "B.Cu") (net 2))
   (segment (start 24.892 98.806) (end 17.018 90.932) (width 0.25) (layer "B.Cu") (net 2))
   (segment (start 41.7625 95.92) (end 41.7625 98.1915) (width 0.25) (layer "B.Cu") (net 2))
@@
   (segment (start 27.432 59.436) (end 26.924 59.944) (width 0.25) (layer "B.Cu") (net 2))
   (segment (start 17.018 76.454) (end 17.018 76.2) (width 0.25) (layer "B.Cu") (net 2))
+  (segment (start 25.0935 114.97) (end 25.0935 116.6385) (width 0.25) (layer "B.Cu") (net 2))
   (segment (start 8.382 22.606) (end 35.814 22.606) (width 0.25) (layer "B.Cu") (net 2))
   (segment (start 7.112 23.876) (end 8.382 22.606) (width 0.25) (layer "B.Cu") (net 2))
@@
   (segment (start 285.496 59.69) (end 292.608 59.69) (width 0.25) (layer "B.Cu") (net 19))
   (segment (start 322.75 19.72) (end 322.75 21.42) (width 0.25) (layer "B.Cu") (net 19))
-  (segment (start 293.37 99.568) (end 293.37 116.332) (width 0.25) (layer "B.Cu") (net 19))
   (segment (start 303.7 117.178) (end 303.022 117.856) (width 0.25) (layer "B.Cu") (net 19))
   (segment (start 303.022 23.368) (end 297.688 23.368) (width 0.25) (layer "B.Cu") (net 19))
+  (segment (start 303.7 97.706) (end 302.6 98.806) (width 0.25) (layer "B.Cu") (net 19))
   (segment (start 293.37 60.706) (end 293.37 60.96) (width 0.25) (layer "B.Cu") (net 19))
   (segment (start 294.386 59.69) (end 293.37 60.706) (width 0.25) (layer "B.Cu") (net 19))
@@
   (segment (start 320.802 23.368) (end 303.022 23.368) (width 0.25) (layer "B.Cu") (net 19))
   (segment (start 303.7 58.504) (end 302.514 59.69) (width 0.25) (layer "B.Cu") (net 19))
-  (segment (start 293.37 116.332) (end 293.624 116.586) (width 0.25) (layer "B.Cu") (net 19))
   (segment (start 292.516 38.77) (end 293.37 39.624) (width 0.25) (layer "B.Cu") (net 19))
   (segment (start 320.548 117.856) (end 322.75 115.654) (width 0.25) (layer "B.Cu") (net 19))
   (segment (start 293.37 39.624) (end 293.37 60.452) (width 0.25) (layer "B.Cu") (net 19))
+  (segment (start 294.132 98.806) (end 293.37 99.568) (width 0.25) (layer "B.Cu") (net 19))
   (segment (start 303.7 39.708) (end 303.022 40.386) (width 0.25) (layer "B.Cu") (net 19))
   (segment (start 284.65 114.97) (end 292.008 114.97) (width 0.25) (layer "B.Cu") (net 19))
   (segment (start 302.514 59.69) (end 294.386 59.69) (width 0.25) (layer "B.Cu") (net 19))
   (segment (start 292.608 59.69) (end 293.37 60.452) (width 0.25) (layer "B.Cu") (net 19))
+  (segment (start 303.7 95.92) (end 303.7 97.706) (width 0.25) (layer "B.Cu") (net 19))
   (segment (start 341.8 76.87) (end 341.8 78.316) (width 0.25) (layer "B.Cu") (net 19))
+  (segment (start 293.37 99.568) (end 293.37 116.332) (width 0.25) (layer "B.Cu") (net 19))
   (segment (start 293.37 80.01) (end 293.37 80.518) (width 0.25) (layer "B.Cu") (net 19))
   (segment (start 293.37 60.452) (end 293.37 60.96) (width 0.25) (layer "B.Cu") (net 19))
@@
   (segment (start 293.37 80.518) (end 293.37 99.568) (width 0.25) (layer "B.Cu") (net 19))
   (segment (start 303.022 40.386) (end 294.132 40.386) (width 0.25) (layer "B.Cu") (net 19))
+  (segment (start 302.6 98.806) (end 294.132 98.806) (width 0.25) (layer "B.Cu") (net 19))
   (segment (start 322.75 21.42) (end 320.802 23.368) (width 0.25) (layer "B.Cu") (net 19))
   (segment (start 294.894 117.856) (end 303.022 117.856) (width 0.25) (layer "B.Cu") (net 19))
@@
   (segment (start 284.65 58.844) (end 285.496 59.69) (width 0.25) (layer "B.Cu") (net 19))
   (segment (start 341.8 78.316) (end 341.122 78.994) (width 0.25) (layer "B.Cu") (net 19))
+  (segment (start 293.37 116.332) (end 293.624 116.586) (width 0.25) (layer "B.Cu") (net 19))
   (segment (start 396.953 69.342) (end 388.874 69.342) (width 0.25) (layer "B.Cu") (net 20))
   (segment (start 387.858 42.418) (end 387.858 62.23) (width 0.25) (layer "B.Cu") (net 20))
@@
   (segment (start 374.65 112.52) (end 374.65 107.315) (width 0.25) (layer "B.Cu") (net 171))
   (segment (start 377.1 114.97) (end 374.65 112.52) (width 0.25) (layer "B.Cu") (net 171))
-  (segment (start 24.384 117.348) (end 12.954 117.348) (width 0.25) (layer "B.Cu") (net 172))
-  (segment (start 25.0935 116.6385) (end 24.384 117.348) (width 0.25) (layer "B.Cu") (net 172))
-  (segment (start 25.0935 114.97) (end 25.0935 116.6385) (width 0.25) (layer "B.Cu") (net 172))
-  (segment (start 303.7 97.706) (end 302.6 98.806) (width 0.25) (layer "B.Cu") (net 173))
-  (segment (start 303.7 95.92) (end 303.7 97.706) (width 0.25) (layer "B.Cu") (net 173))
-  (segment (start 302.6 98.806) (end 294.132 98.806) (width 0.25) (layer "B.Cu") (net 173))
 )

Commit message: component rough layout
Parts:
- added C1: 10p, Capacitor_SMD:C_0402_1005Metric, F.Cu at (83.9, 163.9)
- added C10: 10n, Capacitor_SMD:C_0402_1005Metric, F.Cu at (85.7, 162.9)
- added C11: 1u, Capacitor_SMD:C_0402_1005Metric, F.Cu at (90.2, 164.5)
- added C12: 22u, Capacitor_SMD:C_0805_2012Metric, F.Cu at (91.0, 135.5)
- added C13: 22u, Capacitor_SMD:C_0805_2012Metric, F.Cu at (85.5, 140.3)
- added C2: 10u, Capacitor_SMD:C_0603_1608Metric, F.Cu at (74.2, 162.6)
- added C3: 100n, Capacitor_SMD:C_0402_1005Metric, F.Cu at (79.3, 163.0)
- added C4: 100n, Capacitor_SMD:C_0402_1005Metric, F.Cu at (80.3, 148.0)
- added C5: 100n, Capacitor_SMD:C_0402_1005Metric, F.Cu at (91.3, 151.7)
- added C6: 100n, Capacitor_SMD:C_0402_1005Metric, F.Cu at (91.1, 161.1)
- added C7: 10p, Capacitor_SMD:C_0402_1005Metric, F.Cu at (81.4, 163.9)
- added C8: 100n, Capacitor_SMD:C_0402_1005Metric, F.Cu at (76.3, 159.0)
- added C9: 100n, Capacitor_SMD:C_0402_1005Metric, F.Cu at (91.3, 158.5)
- added H1: MountingHole, MountingHole:MountingHole_2.2mm_M2, F.Cu at (60.7, 122.6)
- added H10: MountingHole, MountingHole:MountingHole_2.2mm_M2, F.Cu at (522.3, 199.0)
- added H11: MountingHole, MountingHole:MountingHole_2.2mm_M2, F.Cu at (376.8, 123.2)
- added H12: MountingHole, MountingHole:MountingHole_2.2mm_M2, F.Cu at (516.8, 121.3)
- added H13: MountingHole, MountingHole:MountingHole_2.2mm_M2, F.Cu at (202.5, 120.2)
- added H14: MountingHole, MountingHole:MountingHole_2.2mm_M2, F.Cu at (103.3, 121.3)
- added H2: MountingHole, MountingHole:MountingHole_2.2mm_M2, F.Cu at (292.8, 250.6)
- added H3: MountingHole, MountingHole:MountingHole_2.2mm_M2, F.Cu at (434.1, 245.1)
- added H4: MountingHole, MountingHole:MountingHole_2.2mm_M2, F.Cu at (175.2, 249.1)
- added H5: MountingHole, MountingHole:MountingHole_2.2mm_M2, F.Cu at (516.1, 245.3)
- added H6: MountingHole, MountingHole:MountingHole_2.2mm_M2, F.Cu at (60.6, 164.3)
- added H7: MountingHole, MountingHole:MountingHole_2.2mm_M2, F.Cu at (89.9, 186.1)
- added H8: MountingHole, MountingHole:MountingHole_2.2mm_M2, F.Cu at (105.2, 246.6)
- added H9: MountingHole, MountingHole:MountingHole_2.2mm_M2, F.Cu at (522.3, 162.6)
- added J1: USB_B_Micro, Connector_USB:USB_Micro-B_Wuerth_629105150521, F.Cu at (94.8, 130.0)
- added J2: SWD, Connector_PinHeader_2.54mm:PinHeader_1x04_P2.54mm_Vertical, F.Cu at (68.1, 140.4)
- added J3: pwr_led+, Connector_PinHeader_2.54mm:PinHeader_1x01_P2.54mm_Vertical, F.Cu at (70.6, 128.8)
- added J4: pwr_led-, Connector_PinHeader_2.54mm:PinHeader_1x01_P2.54mm_Vertical, F.Cu at (75.2, 128.6)
- added J5: caps_led+, Connector_PinHeader_2.54mm:PinHeader_1x01_P2.54mm_Vertical, F.Cu at (72.9, 138.3)
- added J6: caps_led-, Connector_PinHeader_2.54mm:PinHeader_1x01_P2.54mm_Vertical, F.Cu at (73.0, 143.6)
- added R1: 10k, Resistor_SMD:R_0402_1005Metric, F.Cu at (74.3, 157.1)
- added R2: 1k5, Resistor_SMD:R_0603_1608Metric, F.Cu at (95.7, 136.3)
- added R3: 1k5, Resistor_SMD:R_0603_1608Metric, F.Cu at (77.7, 143.5)
- added R4: 1k5, Resistor_SMD:R_0603_1608Metric, F.Cu at (71.1, 133.4)
- added Y1: 16MGz, Crystal:Crystal_SMD_3225-4Pin_3.2x2.5mm, F.Cu at (82.0, 166.6)
- moved U1 370.6 mm to (85.2, 135.5), turned to 180 degrees
- moved MCU1 367.5 mm to (83.8, 155.5), turned to 90 degrees
- moved D1 164.2 mm to (109.4, 139.9)
- moved D10 164.2 mm to (152.3, 216.1)
- moved D100 164.2 mm to (471.4, 197.0)
- moved D101 164.2 mm to (490.4, 197.0)
- moved D102 164.2 mm to (471.4, 216.1)
- moved D103 164.2 mm to (452.3, 216.1)
- moved D104 164.2 mm to (461.9, 235.1)
- moved D105 164.2 mm to (490.4, 139.9)
- moved D106 164.2 mm to (509.5, 139.9)
- moved D107 164.2 mm to (471.4, 158.9)
- moved D108 164.2 mm to (490.4, 158.9)
- moved D109 164.2 mm to (471.4, 178.0)
- moved D11 164.2 mm to (111.8, 235.1)
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Connections:
- D1 pad 2: COLUMN8 -> COLUMN10
- D10 pad 2: COLUMN8 -> COLUMN10
- D100 pad 2: Net-(D100-Pad2) -> COLUMN2
- D101 pad 2: Net-(D100-Pad2) -> COLUMN2
- D102 pad 2: Net-(D100-Pad2) -> COLUMN2
- D103 pad 2: Net-(D100-Pad2) -> COLUMN2
- D104 pad 2: Net-(D100-Pad2) -> COLUMN2
- D11 pad 2: COLUMN8 -> COLUMN10
- D12 pad 2: COLUMN8 -> COLUMN10
- D13 pad 2: Net-(D13-Pad2) -> COLUMN9
- D14 pad 2: Net-(D13-Pad2) -> COLUMN9
- D15 pad 2: Net-(D13-Pad2) -> COLUMN9
- D16 pad 2: Net-(D13-Pad2) -> COLUMN9
- D17 pad 2: Net-(D13-Pad2) -> COLUMN9
- D18 pad 2: Net-(D13-Pad2) -> COLUMN9
- D19 pad 2: Net-(D13-Pad2) -> COLUMN9
- D2 pad 2: COLUMN8 -> COLUMN10
- D20 pad 2: Net-(D13-Pad2) -> COLUMN9
- D21 pad 2: Net-(D13-Pad2) -> COLUMN9
- D22 pad 2: Net-(D13-Pad2) -> COLUMN9
- D23 pad 2: Net-(D13-Pad2) -> COLUMN9
- D24 pad 2: Net-(D13-Pad2) -> COLUMN9
- D25 pad 2: COLUMN7 -> COLUMN8
- D26 pad 2: COLUMN7 -> COLUMN8
- D27 pad 2: COLUMN7 -> COLUMN8
- D28 pad 2: COLUMN7 -> COLUMN8
- D29 pad 2: COLUMN7 -> COLUMN8
- D3 pad 2: COLUMN8 -> COLUMN10
- D30 pad 2: COLUMN7 -> COLUMN8
- D31 pad 2: COLUMN7 -> COLUMN8
- D32 pad 2: COLUMN7 -> COLUMN8
- D33 pad 2: COLUMN7 -> COLUMN8
- D34 pad 2: COLUMN7 -> COLUMN8
- D35 pad 2: COLUMN7 -> COLUMN8
- D36 pad 2: COLUMN7 -> COLUMN8
- D37 pad 2: COLUMN6 -> COLUMN7
- D38 pad 2: COLUMN6 -> COLUMN7
- D39 pad 2: COLUMN6 -> COLUMN7
- D4 pad 2: COLUMN8 -> COLUMN10
- D40 pad 2: COLUMN6 -> COLUMN7
- D41 pad 2: COLUMN6 -> COLUMN7
- D42 pad 2: COLUMN6 -> COLUMN7
- D43 pad 2: COLUMN6 -> COLUMN7
- D44 pad 2: COLUMN6 -> COLUMN7
- D45 pad 2: COLUMN6 -> COLUMN7
- D46 pad 2: COLUMN6 -> COLUMN7
- D47 pad 2: COLUMN6 -> COLUMN7
- D48 pad 2: COLUMN6 -> COLUMN7
- D49 pad 2: COLUMN5 -> COLUMN6
- D5 pad 2: COLUMN8 -> COLUMN10
- D50 pad 2: COLUMN5 -> COLUMN6
- D51 pad 2: COLUMN5 -> COLUMN6
- D52 pad 2: COLUMN5 -> COLUMN6
- D53 pad 2: COLUMN5 -> COLUMN6
- D54 pad 2: COLUMN5 -> COLUMN6
- D55 pad 2: COLUMN5 -> COLUMN6
- D56 pad 2: COLUMN5 -> COLUMN6
- D57 pad 2: COLUMN5 -> COLUMN6
- D58 pad 2: COLUMN5 -> COLUMN6
- D59 pad 2: COLUMN5 -> COLUMN6
- D6 pad 2: COLUMN8 -> COLUMN10
- D60 pad 2: COLUMN5 -> COLUMN6
- D61 pad 2: COLUMN4 -> COLUMN5
- D62 pad 2: COLUMN4 -> COLUMN5
- D63 pad 2: COLUMN4 -> COLUMN5
- D64 pad 2: COLUMN4 -> COLUMN5
- D65 pad 2: COLUMN4 -> COLUMN5
- D66 pad 2: COLUMN4 -> COLUMN5
- D67 pad 2: COLUMN4 -> COLUMN5
- D68 pad 2: COLUMN4 -> COLUMN5
- D69 pad 2: COLUMN4 -> COLUMN5
- D7 pad 2: COLUMN8 -> COLUMN10
- D70 pad 2: COLUMN4 -> COLUMN5
- D71 pad 2: COLUMN4 -> COLUMN5
- D72 pad 2: COLUMN4 -> COLUMN5
- D73 pad 2: COLUMN3 -> COLUMN4
- D74 pad 2: COLUMN3 -> COLUMN4
- D75 pad 2: COLUMN3 -> COLUMN4
- D76 pad 2: COLUMN3 -> COLUMN4
- D77 pad 2: COLUMN3 -> COLUMN4
- D78 pad 2: COLUMN3 -> COLUMN4
- D79 pad 2: COLUMN3 -> COLUMN4
- D8 pad 2: COLUMN8 -> COLUMN10
- D80 pad 2: COLUMN3 -> COLUMN4
- D81 pad 2: COLUMN3 -> COLUMN4
- D82 pad 2: COLUMN3 -> COLUMN4
- D83 pad 2: COLUMN2 -> COLUMN3
- D84 pad 2: COLUMN2 -> COLUMN3
- D85 pad 2: COLUMN2 -> COLUMN3
- D86 pad 2: COLUMN2 -> COLUMN3
- D87 pad 2: COLUMN2 -> COLUMN3
- D88 pad 2: COLUMN2 -> COLUMN3
- D89 pad 2: COLUMN2 -> COLUMN3
- D9 pad 2: COLUMN8 -> COLUMN10
- D90 pad 2: COLUMN2 -> COLUMN3
- D91 pad 2: COLUMN2 -> COLUMN3
- D92 pad 2: COLUMN2 -> COLUMN3
- D93 pad 2: COLUMN2 -> COLUMN3
- D94 pad 2: Net-(D100-Pad2) -> COLUMN2
- D95 pad 2: Net-(D100-Pad2) -> COLUMN2
- D96 pad 2: Net-(D100-Pad2) -> COLUMN2
- D97 pad 2: Net-(D100-Pad2) -> COLUMN2
- D98 pad 2: Net-(D100-Pad2) -> COLUMN2
- D99 pad 2: Net-(D100-Pad2) -> COLUMN2
- MCU1 pad 14: unconnected-(MCU1-Pad14) -> COLUMN10
- MCU1 pad 15: unconnected-(MCU1-Pad15) -> COLUMN9
Routing:
- net COLUMN10: track 0.00 -> 290.1 mm
- net COLUMN9: track 0.00 -> 256.8 mm
- net Net-(D13-Pad2): track 256.8 -> 0.00 mm
- net Net-(D100-Pad2): track 241.3 -> 0.00 mm
- net COLUMN4: track 321.4 -> 268.5 mm
- net COLUMN5: track 282.5 -> 321.4 mm
- net COLUMN2: track 278.2 -> 241.3 mm
- net COLUMN8: track 290.1 -> 270.6 mm
- net ROW2: track 489.8 -> 471.9 mm
- net COLUMN6: track 267.9 -> 282.5 mm
- net COLUMN3: track 268.5 -> 278.2 mm
- net COLUMN7: track 270.6 -> 267.9 mm

Commit message: getting close to pcb first draft
Parts:
- removed H1, H10, H11, H12, H13, H14, H2, H3, H4, H5, H6, H7, H8, H9: MountingHole, MountingHole:MountingHole_2.2mm_M2
- R2: footprint Resistor_SMD:R_0603_1608Metric -> Resistor_SMD:R_0402_1005Metric
- moved C6 15.2 mm to (76.7, 156.4), turned to 180 degrees
- moved R2 12.9 mm to (82.9, 135.3), turned to 180 degrees
- moved C13 12.2 mm to (91.4, 129.7), turned to -90 degrees
- moved U1 12.1 mm to (96.2, 130.3), turned to 90 degrees
- moved J1 11.4 mm to (83.5, 128.9)
- moved R4 10.1 mm to (81.2, 134.6)
- moved C2 9.86 mm to (76.9, 153.1)
- moved R1 7.06 mm to (77.9, 151.0)
- moved C11 6.90 mm to (87.5, 158.1), turned to 180 degrees
- moved J6 6.82 mm to (77.2, 138.2)
- moved C5 6.43 mm to (93.3, 145.6)
- moved C1 6.41 mm to (85.5, 157.7)
- moved C7 6.37 mm to (83.0, 157.8)
- moved C8 6.24 mm to (78.3, 153.1)
- moved MCU1 6.24 mm to (85.8, 149.6)
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Connections:
- net /USB_DM renamed /USB_DN
Routing:
- net COLUMN1: track 231.9 -> 632.2 mm, vias 0 -> 3
- net COLUMN2: track 241.3 -> 600.4 mm, vias 0 -> 3
- net COLUMN3: track 278.2 -> 599.4 mm, vias 0 -> 3
- net COLUMN4: track 268.5 -> 538.5 mm, vias 0 -> 3
- net COLUMN5: track 321.4 -> 550.2 mm, vias 0 -> 3
- net COLUMN6: track 282.5 -> 475.9 mm, vias 0 -> 3
- net COLUMN7: track 267.9 -> 429.8 mm, vias 0 -> 3
- net ROW2: track 471.9 -> 619.0 mm
- net ROW8: track 491.6 -> 635.7 mm
- net ROW10: track 497.7 -> 639.3 mm
- net COLUMN8: track 270.6 -> 395.9 mm, vias 0 -> 3
- net +3.3V: track 0.00 -> 109.2 mm
- net COLUMN9: track 256.8 -> 365.0 mm, vias 0 -> 3
- net ROW12: track 509.3 -> 607.6 mm
- net ROW6: track 517.0 -> 602.4 mm
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- added copper zone on B.Cu, net GND
Other:
- board outline added: 507 x 222 mm

Commit message: Some cleanup
Parts:
- moved R2 0.98 mm to (82.9, 136.3)
- moved Y1 0.48 mm to (83.9, 160.2)
- moved R3 0.45 mm to (80.8, 138.6)
- moved R4 0.44 mm to (80.8, 134.8)
- moved C7 0.33 mm to (83.4, 157.7)
Routing:
- net CAPS_LOCK_LED: track 0.00 -> 37.0 mm, vias 0 -> 2
- net +3.3V: track 109.2 -> 136.6 mm, vias 0 -> 2
- net ROW12: track 607.6 -> 589.5 mm
- net ROW11: track 509.6 -> 495.1 mm
- net ROW9: track 529.7 -> 516.7 mm
- net GND: track 31.0 -> 43.9 mm, vias 12 -> 20
- net ROW8: track 635.7 -> 627.1 mm
- net ROW10: track 639.3 -> 631.2 mm
- net COLUMN9: track 365.0 -> 360.9 mm
- net ROW7: track 547.6 -> 544.0 mm
- net COLUMN10: track 349.7 -> 346.5 mm
- net ROW6: track 602.4 -> 605.4 mm
- net COLUMN3: track 599.4 -> 601.6 mm
- net COLUMN4: track 538.5 -> 540.8 mm
- net COLUMN6: track 475.9 -> 477.8 mm
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
Commit message: Setup edges, starting DRC fixes
Parts:
- moved J1 30.3 mm to (107.8, 110.9)
- moved C13 29.5 mm to (115.8, 113.0)
- moved C3 28.7 mm to (105.3, 141.9)
- moved C8 28.7 mm to (102.7, 137.9)
- moved MCU1 28.7 mm to (110.2, 134.4)
- moved Y1 28.7 mm to (108.3, 145.1)
- moved C4 28.7 mm to (106.1, 127.0)
- moved R2 28.7 mm to (107.2, 121.2)
- moved R4 28.7 mm to (105.2, 119.7)
- moved C1 28.7 mm to (109.9, 142.6)
- moved C10 28.7 mm to (111.9, 141.9)
- moved C11 28.7 mm to (111.9, 143.0)
- moved C12 28.7 mm to (120.5, 121.0)
- moved C2 28.7 mm to (101.2, 138.0)
- moved C5 28.7 mm to (117.7, 130.5)
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Routing:
- net +3.3V: track 136.6 -> 141.3 mm
- net COLUMN9: track 360.9 -> 364.6 mm
- net /USB_DN: track 13.1 -> 16.1 mm
- net /USB_DP: track 13.1 -> 16.1 mm
- net COLUMN8: track 395.6 -> 398.0 mm
- net COLUMN7: track 430.1 -> 432.4 mm
- net COLUMN10: track 346.5 -> 348.9 mm
- net ROW9: track 516.7 -> 518.8 mm
- net ROW6: track 605.4 -> 607.5 mm
- net ROW5: track 455.0 -> 457.1 mm
- net ROW11: track 495.1 -> 497.2 mm
- net ROW10: track 631.2 -> 633.3 mm
- net COLUMN1: track 634.1 -> 636.2 mm
- net ROW4: track 593.2 -> 595.3 mm
- net ROW12: track 589.5 -> 591.6 mm
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Other:
- board size 507 x 222 mm -> 458 x 143.5 mm

Commit message: Get rid of need for key signals on left side of board
Parts:
- moved J1 0.20 mm to (107.8, 111.1)
- moved C5 0.20 mm to (117.8, 130.5)
Connections:
- MCU1 pad 15: COLUMN9 -> ROW12
- MCU1 pad 16: COLUMN8 -> ROW11
- MCU1 pad 17: COLUMN7 -> ROW10
- MCU1 pad 20: COLUMN6 -> ROW9
- MCU1 pad 21: COLUMN5 -> ROW8
- MCU1 pad 22: COLUMN4 -> ROW7
- MCU1 pad 23: COLUMN3 -> ROW6
- MCU1 pad 24: COLUMN2 -> ROW5
- MCU1 pad 25: COLUMN1 -> COLUMN9
- MCU1 pad 27: ROW12 -> COLUMN8
- MCU1 pad 28: ROW11 -> COLUMN7
- MCU1 pad 29: ROW10 -> COLUMN6
- MCU1 pad 30: ROW9 -> COLUMN5
- MCU1 pad 33: ROW8 -> COLUMN4
- MCU1 pad 34: ROW7 -> COLUMN3
- MCU1 pad 35: ROW6 -> COLUMN2
- MCU1 pad 36: ROW5 -> COLUMN1
Routing:
- net ROW5: track 457.1 -> 442.4 mm
- net ROW6: track 607.5 -> 595.1 mm
- net ROW7: track 545.4 -> 533.6 mm
- net ROW8: track 629.2 -> 618.4 mm
- net ROW9: track 518.8 -> 529.6 mm
- net COLUMN1: track 636.2 -> 645.3 mm, vias 3 -> 1
- net ROW10: track 633.3 -> 624.4 mm
- net COLUMN2: track 604.4 -> 611.8 mm, vias 3 -> 1
- net ROW11: track 497.2 -> 490.2 mm
- net ROW12: track 591.6 -> 585.2 mm
- net COLUMN3: track 603.7 -> 610.1 mm, vias 3 -> 1
- net COLUMN4: track 542.9 -> 547.7 mm, vias 3 -> 1
- net COLUMN9: track 364.6 -> 361.4 mm, vias 3 -> 1
- net COLUMN8: track 398.0 -> 395.6 mm, vias 3 -> 1
- net COLUMN7: track 432.4 -> 431.2 mm, vias 3 -> 1
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
Commit message: little more trace cleanup
Routing:
- net COLUMN8: track 395.6 -> 392.7 mm
- net COLUMN7: track 431.2 -> 428.3 mm
- net COLUMN6: track 479.3 -> 476.4 mm
- net COLUMN5: track 554.3 -> 551.4 mm
- net COLUMN4: track 547.7 -> 544.8 mm
- net COLUMN3: track 610.1 -> 607.2 mm
- net COLUMN2: track 611.8 -> 608.9 mm
- net COLUMN9: track 361.4 -> 358.5 mm
- net COLUMN1: track 645.3 -> 642.4 mm
