File: kicad/kicad.kicad_pcb (KiCad board)
At the start: 2 copper layers, 458 x 143.5 mm, 256 parts, among them J1 USB_B_Micro, J2 SWD, J3 pwr_led+, J4 pwr_led-, J5 caps_led+, J6 caps_led-, U1 AMS1117-3.3, Y1 16MGz, sw1 Esc, sw10 Z, sw100 N5, sw101 N6, sw102 N2, sw103 N1, sw104 N0, sw105 MPlay, sw106 MFwd, sw107 NSlash, sw108 NStar, sw109 N8, sw11 LCtrl, sw110 N9, sw111 NMinus, sw112 NPlus, sw113 NEnter, sw114 N3, sw115 NPeriod, sw12 LSys, sw13 F2, sw14 F3, sw15 2, sw16 3, sw17 W, sw18 E, sw19 S, sw2 F1, sw20 D, sw21 X, sw22 C, sw23 LAlt, sw24 THome, sw25 F4, sw26 F5, sw27 4, sw28 5, sw29 R, sw3 Tilda, sw30 T, sw31 F, sw32 G, sw33 V, sw34 B, sw35 LSpace, sw36 TLeft, sw37 F6, sw38 F7, sw39 6, sw4 1, sw40 7, sw41 Y, sw42 U, sw43 H, sw44 J, sw45 N, sw46 M, sw47 TUp, sw48 TDown, sw49 F8, sw5 Tab, sw50 F9, sw51 8, sw52 9, sw53 I, sw54 O, sw55 K, sw56 L, sw57 Comma, sw58 Period, sw59 RSpace, sw6 Q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

Commit message: layout new diodes
Parts:
- D1: value D-Esc -> 1N4148W; footprint Diode_SMD:D_SOD-123F -> Diode_SMD:D_SOD-123
- D10: value D-Z -> 1N4148W; footprint Diode_SMD:D_SOD-123F -> Diode_SMD:D_SOD-123
- D100: value D-Num5 -> 1N4148W; footprint Diode_SMD:D_SOD-123F -> Diode_SMD:D_SOD-123
- D101: value D-Num6 -> 1N4148W; footprint Diode_SMD:D_SOD-123F -> Diode_SMD:D_SOD-123
- D102: value D-Num2 -> 1N4148W; footprint Diode_SMD:D_SOD-123F -> Diode_SMD:D_SOD-123
- D103: value D-Num1 -> 1N4148W; footprint Diode_SMD:D_SOD-123F -> Diode_SMD:D_SOD-123
- D104: value D-Num0 -> 1N4148W; footprint Diode_SMD:D_SOD-123F -> Diode_SMD:D_SOD-123
- D105: value D-mPlay -> 1N4148W; footprint Diode_SMD:D_SOD-123F -> Diode_SMD:D_SOD-123
- D106: value D-mFwd -> 1N4148W; footprint Diode_SMD:D_SOD-123F -> Diode_SMD:D_SOD-123
- D107: value D-Num/ -> 1N4148W; footprint Diode_SMD:D_SOD-123F -> Diode_SMD:D_SOD-123
- D108: value D-Num* -> 1N4148W; footprint Diode_SMD:D_SOD-123F -> Diode_SMD:D_SOD-123
- D109: value D-Num8 -> 1N4148W; footprint Diode_SMD:D_SOD-123F -> Diode_SMD:D_SOD-123
- D11: value D-LCtrl -> 1N4148W; footprint Diode_SMD:D_SOD-123F -> Diode_SMD:D_SOD-123
- D110, D99: value D-Num9 -> 1N4148W; footprint Diode_SMD:D_SOD-123F -> Diode_SMD:D_SOD-123
- D111: value D-Num- -> 1N4148W; footprint Diode_SMD:D_SOD-123F -> Diode_SMD:D_SOD-123
- D112: value D-Num+ -> 1N4148W; footprint Diode_SMD:D_SOD-123F -> Diode_SMD:D_SOD-123
- D113: value D-NumEnter -> 1N4148W; footprint Diode_SMD:D_SOD-123F -> Diode_SMD:D_SOD-123
- D114: value D-Num3 -> 1N4148W; footprint Diode_SMD:D_SOD-123F -> Diode_SMD:D_SOD-123
- D115: value D-Num. -> 1N4148W; footprint Diode_SMD:D_SOD-123F -> Diode_SMD:D_SOD-123
- D12: value D-LSys -> 1N4148W; footprint Diode_SMD:D_SOD-123F -> Diode_SMD:D_SOD-123
- D13: value D-F2 -> 1N4148W; footprint Diode_SMD:D_SOD-123F -> Diode_SMD:D_SOD-123
- D14: value D-F3 -> 1N4148W; footprint Diode_SMD:D_SOD-123F -> Diode_SMD:D_SOD-123
- D15: value D-2 -> 1N4148W; footprint Diode_SMD:D_SOD-123F -> Diode_SMD:D_SOD-123
- D16: value D-3 -> 1N4148W; footprint Diode_SMD:D_SOD-123F -> Diode_SMD:D_SOD-123
- D17: value D-W -> 1N4148W; footprint Diode_SMD:D_SOD-123F -> Diode_SMD:D_SOD-123
- D18: value D-E -> 1N4148W; footprint Diode_SMD:D_SOD-123F -> Diode_SMD:D_SOD-123
- D19: value D-S -> 1N4148W; footprint Diode_SMD:D_SOD-123F -> Diode_SMD:D_SOD-123
- D2: value D-F1 -> 1N4148W; footprint Diode_SMD:D_SOD-123F -> Diode_SMD:D_SOD-123
- D20: value D-D -> 1N4148W; footprint Diode_SMD:D_SOD-123F -> Diode_SMD:D_SOD-123
- D21: value D-X -> 1N4148W; footprint Diode_SMD:D_SOD-123F -> Diode_SMD:D_SOD-123
- D22: value D-C -> 1N4148W; footprint Diode_SMD:D_SOD-123F -> Diode_SMD:D_SOD-123
- D23: value D-LAlt -> 1N4148W; footprint Diode_SMD:D_SOD-123F -> Diode_SMD:D_SOD-123
- D24: value D-THome -> 1N4148W; footprint Diode_SMD:D_SOD-123F -> Diode_SMD:D_SOD-123
- D25: value D-F4 -> 1N4148W; footprint Diode_SMD:D_SOD-123F -> Diode_SMD:D_SOD-123
- D26: value D-F5 -> 1N4148W; footprint Diode_SMD:D_SOD-123F -> Diode_SMD:D_SOD-123
- D27: value D-4 -> 1N4148W; footprint Diode_SMD:D_SOD-123F -> Diode_SMD:D_SOD-123
- D28: value D-5 -> 1N4148W; footprint Diode_SMD:D_SOD-123F -> Diode_SMD:D_SOD-123
- D29: value D-R -> 1N4148W; footprint Diode_SMD:D_SOD-123F -> Diode_SMD:D_SOD-123
- D3: value D-Tilda -> 1N4148W; footprint Diode_SMD:D_SOD-123F -> Diode_SMD:D_SOD-123
- D30: value D-T -> 1N4148W; footprint Diode_SMD:D_SOD-123F -> Diode_SMD:D_SOD-123
- D31: value D-F -> 1N4148W; footprint Diode_SMD:D_SOD-123F -> Diode_SMD:D_SOD-123
- D32: value D-G -> 1N4148W; footprint Diode_SMD:D_SOD-123F -> Diode_SMD:D_SOD-123
- D33: value D-V -> 1N4148W; footprint Diode_SMD:D_SOD-123F -> Diode_SMD:D_SOD-123
- D34: value D-B -> 1N4148W; footprint Diode_SMD:D_SOD-123F -> Diode_SMD:D_SOD-123
- D35: value D-LSpace -> 1N4148W; footprint Diode_SMD:D_SOD-123F -> Diode_SMD:D_SOD-123
- D36: value D-TLeft -> 1N4148W; footprint Diode_SMD:D_SOD-123F -> Diode_SMD:D_SOD-123
- D37: value D-F6 -> 1N4148W; footprint Diode_SMD:D_SOD-123F -> Diode_SMD:D_SOD-123
- D38: value D-F7 -> 1N4148W; footprint Diode_SMD:D_SOD-123F -> Diode_SMD:D_SOD-123
- D39: value D-6 -> 1N4148W; footprint Diode_SMD:D_SOD-123F -> Diode_SMD:D_SOD-123
- D4: value D-1 -> 1N4148W; footprint Diode_SMD:D_SOD-123F -> Diode_SMD:D_SOD-123
- D40: value D-7 -> 1N4148W; footprint Diode_SMD:D_SOD-123F -> Diode_SMD:D_SOD-123
- D41: value D-Y -> 1N4148W; footprint Diode_SMD:D_SOD-123F -> Diode_SMD:D_SOD-123
- D42: value D-U -> 1N4148W; footprint Diode_SMD:D_SOD-123F -> Diode_SMD:D_SOD-123
- D43: value D-H -> 1N4148W; footprint Diode_SMD:D_SOD-123F -> Diode_SMD:D_SOD-123
- D44: value D-J -> 1N4148W; footprint Diode_SMD:D_SOD-123F -> Diode_SMD:D_SOD-123
- D45: value D-N -> 1N4148W; footprint Diode_SMD:D_SOD-123F -> Diode_SMD:D_SOD-123
- D46: value D-M -> 1N4148W; footprint Diode_SMD:D_SOD-123F -> Diode_SMD:D_SOD-123
- D47: value D-TUp -> 1N4148W; footprint Diode_SMD:D_SOD-123F -> Diode_SMD:D_SOD-123
- D48: value D-TDown -> 1N4148W; footprint Diode_SMD:D_SOD-123F -> Diode_SMD:D_SOD-123
- D49: value D-F8 -> 1N4148W; footprint Diode_SMD:D_SOD-123F -> Diode_SMD:D_SOD-123
- D5: value D-Tab -> 1N4148W; footprint Diode_SMD:D_SOD-123F -> Diode_SMD:D_SOD-123
- D50: value D-F9 -> 1N4148W; footprint Diode_SMD:D_SOD-123F -> Diode_SMD:D_SOD-123
- D51: value D-8 -> 1N4148W; footprint Diode_SMD:D_SOD-123F -> Diode_SMD:D_SOD-123
- D52: value D-9 -> 1N4148W; footprint Diode_SMD:D_SOD-123F -> Diode_SMD:D_SOD-123
- D53: value D-I -> 1N4148W; footprint Diode_SMD:D_SOD-123F -> Diode_SMD:D_SOD-123
- D54: value D-O -> 1N4148W; footprint Diode_SMD:D_SOD-123F -> Diode_SMD:D_SOD-123
- D55: value D-K -> 1N4148W; footprint Diode_SMD:D_SOD-123F -> Diode_SMD:D_SOD-123
- D56: value D-L -> 1N4148W; footprint Diode_SMD:D_SOD-123F -> Diode_SMD:D_SOD-123
- D57: value D-, -> 1N4148W; footprint Diode_SMD:D_SOD-123F -> Diode_SMD:D_SOD-123
- D58: value D-. -> 1N4148W; footprint Diode_SMD:D_SOD-123F -> Diode_SMD:D_SOD-123
- D59: value D-RSpace -> 1N4148W; footprint Diode_SMD:D_SOD-123F -> Diode_SMD:D_SOD-123
- D6: value D-Q -> 1N4148W; footprint Diode_SMD:D_SOD-123F -> Diode_SMD:D_SOD-123
- D60: value D-TRight -> 1N4148W; footprint Diode_SMD:D_SOD-123F -> Diode_SMD:D_SOD-123
- D61: value D-F10 -> 1N4148W; footprint Diode_SMD:D_SOD-123F -> Diode_SMD:D_SOD-123
- D62: value D-F11 -> 1N4148W; footprint Diode_SMD:D_SOD-123F -> Diode_SMD:D_SOD-123
- D63: value D-0 -> 1N4148W; footprint Diode_SMD:D_SOD-123F -> Diode_SMD:D_SOD-123
- D64: value D-- -> 1N4148W; footprint Diode_SMD:D_SOD-123F -> Diode_SMD:D_SOD-123
- D65: value D-P -> 1N4148W; footprint Diode_SMD:D_SOD-123F -> Diode_SMD:D_SOD-123
- D66: value D-[ -> 1N4148W; footprint Diode_SMD:D_SOD-123F -> Diode_SMD:D_SOD-123
- D67: value D-; -> 1N4148W; footprint Diode_SMD:D_SOD-123F -> Diode_SMD:D_SOD-123
- D68: value D-' -> 1N4148W; footprint Diode_SMD:D_SOD-123F -> Diode_SMD:D_SOD-123
- D69: value D-/ -> 1N4148W; footprint Diode_SMD:D_SOD-123F -> Diode_SMD:D_SOD-123
- D7: value D-CAPS -> 1N4148W; footprint Diode_SMD:D_SOD-123F -> Diode_SMD:D_SOD-123
- D70: value D-RShift -> 1N4148W; footprint Diode_SMD:D_SOD-123F -> Diode_SMD:D_SOD-123
- D71: value D-RAlt -> 1N4148W; footprint Diode_SMD:D_SOD-123F -> Diode_SMD:D_SOD-123
- D72: value D-TEnd -> 1N4148W; footprint Diode_SMD:D_SOD-123F -> Diode_SMD:D_SOD-123
- D73: value D-F12 -> 1N4148W; footprint Diode_SMD:D_SOD-123F -> Diode_SMD:D_SOD-123
- D74: value D-PrtSc -> 1N4148W; footprint Diode_SMD:D_SOD-123F -> Diode_SMD:D_SOD-123
- D75: value D-= -> 1N4148W; footprint Diode_SMD:D_SOD-123F -> Diode_SMD:D_SOD-123
- D76: value D-BcSpc -> 1N4148W; footprint Diode_SMD:D_SOD-123F -> Diode_SMD:D_SOD-123
- D77: value D-] -> 1N4148W; footprint Diode_SMD:D_SOD-123F -> Diode_SMD:D_SOD-123
- D78: value D-\ -> 1N4148W; footprint Diode_SMD:D_SOD-123F -> Diode_SMD:D_SOD-123
- D79: value D-Enter -> 1N4148W; footprint Diode_SMD:D_SOD-123F -> Diode_SMD:D_SOD-123
- D8: value D-A -> 1N4148W; footprint Diode_SMD:D_SOD-123F -> Diode_SMD:D_SOD-123
- D80: value D-RCtrl -> 1N4148W; footprint Diode_SMD:D_SOD-123F -> Diode_SMD:D_SOD-123
- D81: value D-RSys -> 1N4148W; footprint Diode_SMD:D_SOD-123F -> Diode_SMD:D_SOD-123
- D82: value D-Menu -> 1N4148W; footprint Diode_SMD:D_SOD-123F -> Diode_SMD:D_SOD-123
- D83: value D-ScrLck -> 1N4148W; footprint Diode_SMD:D_SOD-123F -> Diode_SMD:D_SOD-123
- D84: value D-Pause -> 1N4148W; footprint Diode_SMD:D_SOD-123F -> Diode_SMD:D_SOD-123
- D85: value D-Insert -> 1N4148W; footprint Diode_SMD:D_SOD-123F -> Diode_SMD:D_SOD-123
- D86: value D-Home -> 1N4148W; footprint Diode_SMD:D_SOD-123F -> Diode_SMD:D_SOD-123
- D87: value D-Dlt -> 1N4148W; footprint Diode_SMD:D_SOD-123F -> Diode_SMD:D_SOD-123
- D88: value D-End -> 1N4148W; footprint Diode_SMD:D_SOD-123F -> Diode_SMD:D_SOD-123
- D89: value D-Num4 -> 1N4148W; footprint Diode_SMD:D_SOD-123F -> Diode_SMD:D_SOD-123
- D9: value D-LShift -> 1N4148W; footprint Diode_SMD:D_SOD-123F -> Diode_SMD:D_SOD-123
- D90: value D-Up -> 1N4148W; footprint Diode_SMD:D_SOD-123F -> Diode_SMD:D_SOD-123
- D91: value D-Down -> 1N4148W; footprint Diode_SMD:D_SOD-123F -> Diode_SMD:D_SOD-123
- D92: value D-Left -> 1N4148W; footprint Diode_SMD:D_SOD-123F -> Diode_SMD:D_SOD-123
- D93: value D-Right -> 1N4148W; footprint Diode_SMD:D_SOD-123F -> Diode_SMD:D_SOD-123
- D94: value D-FN -> 1N4148W; footprint Diode_SMD:D_SOD-123F -> Diode_SMD:D_SOD-123
- D95: value D-mBack -> 1N4148W; footprint Diode_SMD:D_SOD-123F -> Diode_SMD:D_SOD-123
- D96: value D-PgUp -> 1N4148W; footprint Diode_SMD:D_SOD-123F -> Diode_SMD:D_SOD-123
- D97: value D-NumLck -> 1N4148W; footprint Diode_SMD:D_SOD-123F -> Diode_SMD:D_SOD-123
- D98: value D-PgDwn -> 1N4148W; footprint Diode_SMD:D_SOD-123F -> Diode_SMD:D_SOD-123
- moved D104 38.1 mm to (450.0, 210.9), turned to 180 degrees
- moved D106 38.1 mm to (497.6, 115.7), turned to 180 degrees
- moved D111 38.1 mm to (497.6, 134.8), turned to 180 degrees
- moved D112 38.1 mm to (497.6, 163.3), turned to 180 degrees
- moved D113 38.1 mm to (497.6, 201.4), turned to 180 degrees
- moved D38 38.1 mm to (259.5, 115.7), turned to 180 degrees
- moved D45 38.1 mm to (235.7, 191.9), turned to 180 degrees
- moved D50 38.1 mm to (307.1, 115.7), turned to 180 degrees
- moved D53 38.1 mm to (259.5, 153.8), turned to 180 degrees
- moved D55 38.1 mm to (264.3, 172.8), turned to 180 degrees
- moved D56 38.1 mm to (283.3, 172.8), turned to 180 degrees
- moved D63 38.1 mm to (288.1, 134.8), turned to 180 degrees
- moved D64 38.1 mm to (307.1, 134.8), turned to 180 degrees
- moved D69 38.1 mm to (311.9, 191.9), turned to 180 degrees
- moved D72 38.1 mm to (259.5, 230.0), turned to 180 degrees
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Connections:
- D1 pad 1: Net-(D1-Pad1) -> COLUMN10
- D1 pad 2: COLUMN10 -> Net-(D1-Pad2)
- D10 pad 1: Net-(D10-Pad1) -> COLUMN10
- D10 pad 2: COLUMN10 -> Net-(D10-Pad2)
- D100 pad 1: Net-(D100-Pad1) -> COLUMN2
- D100 pad 2: COLUMN2 -> Net-(D100-Pad2)
- D101 pad 1: Net-(D101-Pad1) -> COLUMN2
- D101 pad 2: COLUMN2 -> Net-(D101-Pad2)
- D102 pad 1: Net-(D102-Pad1) -> COLUMN2
- D102 pad 2: COLUMN2 -> Net-(D102-Pad2)
- D103 pad 1: Net-(D103-Pad1) -> COLUMN2
- D103 pad 2: COLUMN2 -> Net-(D103-Pad2)
- D104 pad 1: Net-(D104-Pad1) -> COLUMN2
- D104 pad 2: COLUMN2 -> Net-(D104-Pad2)
- D105 pad 1: Net-(D105-Pad1) -> COLUMN1
- D105 pad 2: COLUMN1 -> Net-(D105-Pad2)
- D106 pad 1: Net-(D106-Pad1) -> COLUMN1
- D106 pad 2: COLUMN1 -> Net-(D106-Pad2)
- D107 pad 1: Net-(D107-Pad1) -> COLUMN1
- D107 pad 2: COLUMN1 -> Net-(D107-Pad2)
- D108 pad 1: Net-(D108-Pad1) -> COLUMN1
- D108 pad 2: COLUMN1 -> Net-(D108-Pad2)
- D109 pad 1: Net-(D109-Pad1) -> COLUMN1
- D109 pad 2: COLUMN1 -> Net-(D109-Pad2)
- D11 pad 1: Net-(D11-Pad1) -> COLUMN10
- D11 pad 2: COLUMN10 -> Net-(D11-Pad2)
- D110 pad 1: Net-(D110-Pad1) -> COLUMN1
- D110 pad 2: COLUMN1 -> Net-(D110-Pad2)
- D111 pad 1: Net-(D111-Pad1) -> COLUMN1
- D111 pad 2: COLUMN1 -> Net-(D111-Pad2)
- D112 pad 1: Net-(D112-Pad1) -> COLUMN1
- D112 pad 2: COLUMN1 -> Net-(D112-Pad2)
- D113 pad 1: Net-(D113-Pad1) -> COLUMN1
- D113 pad 2: COLUMN1 -> Net-(D113-Pad2)
- D114 pad 1: Net-(D114-Pad1) -> COLUMN1
- D114 pad 2: COLUMN1 -> Net-(D114-Pad2)
- D115 pad 1: Net-(D115-Pad1) -> COLUMN1
- D115 pad 2: COLUMN1 -> Net-(D115-Pad2)
- D12 pad 1: Net-(D12-Pad1) -> COLUMN10
- D12 pad 2: COLUMN10 -> Net-(D12-Pad2)
- D13 pad 1: Net-(D13-Pad1) -> COLUMN9
- D13 pad 2: COLUMN9 -> Net-(D13-Pad2)
- D14 pad 1: Net-(D14-Pad1) -> COLUMN9
- D14 pad 2: COLUMN9 -> Net-(D14-Pad2)
- D15 pad 1: Net-(D15-Pad1) -> COLUMN9
- D15 pad 2: COLUMN9 -> Net-(D15-Pad2)
- D16 pad 1: Net-(D16-Pad1) -> COLUMN9
- D16 pad 2: COLUMN9 -> Net-(D16-Pad2)
- D17 pad 1: Net-(D17-Pad1) -> COLUMN9
- D17 pad 2: COLUMN9 -> Net-(D17-Pad2)
- D18 pad 1: Net-(D18-Pad1) -> COLUMN9
- D18 pad 2: COLUMN9 -> Net-(D18-Pad2)
- D19 pad 1: Net-(D19-Pad1) -> COLUMN9
- D19 pad 2: COLUMN9 -> Net-(D19-Pad2)
- D2 pad 1: Net-(D2-Pad1) -> COLUMN10
- D2 pad 2: COLUMN10 -> Net-(D2-Pad2)
- D20 pad 1: Net-(D20-Pad1) -> COLUMN9
- D20 pad 2: COLUMN9 -> Net-(D20-Pad2)
- D21 pad 1: Net-(D21-Pad1) -> COLUMN9
- D21 pad 2: COLUMN9 -> Net-(D21-Pad2)
- D22 pad 1: Net-(D22-Pad1) -> COLUMN9
- D22 pad 2: COLUMN9 -> Net-(D22-Pad2)
- D23 pad 1: Net-(D23-Pad1) -> COLUMN9
- D23 pad 2: COLUMN9 -> Net-(D23-Pad2)
- D24 pad 1: Net-(D24-Pad1) -> COLUMN9
- D24 pad 2: COLUMN9 -> Net-(D24-Pad2)
- D25 pad 1: Net-(D25-Pad1) -> COLUMN8
- D25 pad 2: COLUMN8 -> Net-(D25-Pad2)
- D26 pad 1: Net-(D26-Pad1) -> COLUMN8
- D26 pad 2: COLUMN8 -> Net-(D26-Pad2)
- D27 pad 1: Net-(D27-Pad1) -> COLUMN8
- D27 pad 2: COLUMN8 -> Net-(D27-Pad2)
- D28 pad 1: Net-(D28-Pad1) -> COLUMN8
- D28 pad 2: COLUMN8 -> Net-(D28-Pad2)
- D29 pad 1: Net-(D29-Pad1) -> COLUMN8
- D29 pad 2: COLUMN8 -> Net-(D29-Pad2)
- D3 pad 1: Net-(D3-Pad1) -> COLUMN10
- D3 pad 2: COLUMN10 -> Net-(D3-Pad2)
- D30 pad 1: Net-(D30-Pad1) -> COLUMN8
- D30 pad 2: COLUMN8 -> Net-(D30-Pad2)
- D31 pad 1: Net-(D31-Pad1) -> COLUMN8
- D31 pad 2: COLUMN8 -> Net-(D31-Pad2)
- D32 pad 1: Net-(D32-Pad1) -> COLUMN8
- D32 pad 2: COLUMN8 -> Net-(D32-Pad2)
- D33 pad 1: Net-(D33-Pad1) -> COLUMN8
- D33 pad 2: COLUMN8 -> Net-(D33-Pad2)
- D34 pad 1: Net-(D34-Pad1) -> COLUMN8
- D34 pad 2: COLUMN8 -> Net-(D34-Pad2)
- D35 pad 1: Net-(D35-Pad1) -> COLUMN8
- D35 pad 2: COLUMN8 -> Net-(D35-Pad2)
- D36 pad 1: Net-(D36-Pad1) -> COLUMN8
- D36 pad 2: COLUMN8 -> Net-(D36-Pad2)
- D37 pad 1: Net-(D37-Pad1) -> COLUMN7
- D37 pad 2: COLUMN7 -> Net-(D37-Pad2)
- D38 pad 1: Net-(D38-Pad1) -> COLUMN7
- D38 pad 2: COLUMN7 -> Net-(D38-Pad2)
- D39 pad 1: Net-(D39-Pad1) -> COLUMN7
- D39 pad 2: COLUMN7 -> Net-(D39-Pad2)
- D4 pad 1: Net-(D4-Pad1) -> COLUMN10
- D4 pad 2: COLUMN10 -> Net-(D4-Pad2)
- D40 pad 1: Net-(D40-Pad1) -> COLUMN7
- D40 pad 2: COLUMN7 -> Net-(D40-Pad2)
- D41 pad 1: Net-(D41-Pad1) -> COLUMN7
- D41 pad 2: COLUMN7 -> Net-(D41-Pad2)
- D42 pad 1: Net-(D42-Pad1) -> COLUMN7
- D42 pad 2: COLUMN7 -> Net-(D42-Pad2)
- D43 pad 1: Net-(D43-Pad1) -> COLUMN7
- D43 pad 2: COLUMN7 -> Net-(D43-Pad2)
- D44 pad 1: Net-(D44-Pad1) -> COLUMN7
- D44 pad 2: COLUMN7 -> Net-(D44-Pad2)
- D45 pad 1: Net-(D45-Pad1) -> COLUMN7
- D45 pad 2: COLUMN7 -> Net-(D45-Pad2)
- D46 pad 1: Net-(D46-Pad1) -> COLUMN7
- D46 pad 2: COLUMN7 -> Net-(D46-Pad2)
- D47 pad 1: Net-(D47-Pad1) -> COLUMN7
- D47 pad 2: COLUMN7 -> Net-(D47-Pad2)
- D48 pad 1: Net-(D48-Pad1) -> COLUMN7
- D48 pad 2: COLUMN7 -> Net-(D48-Pad2)
- D49 pad 1: Net-(D49-Pad1) -> COLUMN6
- D49 pad 2: COLUMN6 -> Net-(D49-Pad2)
- D5 pad 1: Net-(D5-Pad1) -> COLUMN10
- D5 pad 2: COLUMN10 -> Net-(D5-Pad2)
- D50 pad 1: Net-(D50-Pad1) -> COLUMN6
- D50 pad 2: COLUMN6 -> Net-(D50-Pad2)
- D51 pad 1: Net-(D51-Pad1) -> COLUMN6
- D51 pad 2: COLUMN6 -> Net-(D51-Pad2)
- D52 pad 1: Net-(D52-Pad1) -> COLUMN6
- D52 pad 2: COLUMN6 -> Net-(D52-Pad2)
- D53 pad 1: Net-(D53-Pad1) -> COLUMN6
- D53 pad 2: COLUMN6 -> Net-(D53-Pad2)
- D54 pad 1: Net-(D54-Pad1) -> COLUMN6
- D54 pad 2: COLUMN6 -> Net-(D54-Pad2)
- D55 pad 1: Net-(D55-Pad1) -> COLUMN6
- D55 pad 2: COLUMN6 -> Net-(D55-Pad2)
- D56 pad 1: Net-(D56-Pad1) -> COLUMN6
- D56 pad 2: COLUMN6 -> Net-(D56-Pad2)
- D57 pad 1: Net-(D57-Pad1) -> COLUMN6
- D57 pad 2: COLUMN6 -> Net-(D57-Pad2)
- D58 pad 1: Net-(D58-Pad1) -> COLUMN6
- D58 pad 2: COLUMN6 -> Net-(D58-Pad2)
- D59 pad 1: Net-(D59-Pad1) -> COLUMN6
- D59 pad 2: COLUMN6 -> Net-(D59-Pad2)
- D6 pad 1: Net-(D6-Pad1) -> COLUMN10
- D6 pad 2: COLUMN10 -> Net-(D6-Pad2)
- D60 pad 1: Net-(D60-Pad1) -> COLUMN6
- D60 pad 2: COLUMN6 -> Net-(D60-Pad2)
- D61 pad 1: Net-(D61-Pad1) -> COLUMN5
- D61 pad 2: COLUMN5 -> Net-(D61-Pad2)
- D62 pad 1: Net-(D62-Pad1) -> COLUMN5
- D62 pad 2: COLUMN5 -> Net-(D62-Pad2)
- D63 pad 1: Net-(D63-Pad1) -> COLUMN5
- D63 pad 2: COLUMN5 -> Net-(D63-Pad2)
- D64 pad 1: Net-(D64-Pad1) -> COLUMN5
- D64 pad 2: COLUMN5 -> Net-(D64-Pad2)
- D65 pad 1: Net-(D65-Pad1) -> COLUMN5
- D65 pad 2: COLUMN5 -> Net-(D65-Pad2)
- D66 pad 1: Net-(D66-Pad1) -> COLUMN5
- D66 pad 2: COLUMN5 -> Net-(D66-Pad2)
- D67 pad 1: Net-(D67-Pad1) -> COLUMN5
- D67 pad 2: COLUMN5 -> Net-(D67-Pad2)
- D68 pad 1: Net-(D68-Pad1) -> COLUMN5
- D68 pad 2: COLUMN5 -> Net-(D68-Pad2)
- D69 pad 1: Net-(D69-Pad1) -> COLUMN5
- D69 pad 2: COLUMN5 -> Net-(D69-Pad2)
- D7 pad 1: Net-(D7-Pad1) -> COLUMN10
- D7 pad 2: COLUMN10 -> Net-(D7-Pad2)
- D70 pad 1: Net-(D70-Pad1) -> COLUMN5
- D70 pad 2: COLUMN5 -> Net-(D70-Pad2)
- D71 pad 1: Net-(D71-Pad1) -> COLUMN5
- D71 pad 2: COLUMN5 -> Net-(D71-Pad2)
- D72 pad 1: Net-(D72-Pad1) -> COLUMN5
- D72 pad 2: COLUMN5 -> Net-(D72-Pad2)
- D73 pad 1: Net-(D73-Pad1) -> COLUMN4
- D73 pad 2: COLUMN4 -> Net-(D73-Pad2)
- D74 pad 1: Net-(D74-Pad1) -> COLUMN4
- D74 pad 2: COLUMN4 -> Net-(D74-Pad2)
- D75 pad 1: Net-(D75-Pad1) -> COLUMN4
- D75 pad 2: COLUMN4 -> Net-(D75-Pad2)
- D76 pad 1: Net-(D76-Pad1) -> COLUMN4
- D76 pad 2: COLUMN4 -> Net-(D76-Pad2)
- D77 pad 1: Net-(D77-Pad1) -> COLUMN4
- D77 pad 2: COLUMN4 -> Net-(D77-Pad2)
- D78 pad 1: Net-(D78-Pad1) -> COLUMN4
- D78 pad 2: COLUMN4 -> Net-(D78-Pad2)
- D79 pad 1: Net-(D79-Pad1) -> COLUMN4
- D79 pad 2: COLUMN4 -> Net-(D79-Pad2)
- D8 pad 1: Net-(D8-Pad1) -> COLUMN10
- D8 pad 2: COLUMN10 -> Net-(D8-Pad2)
- D80 pad 1: Net-(D80-Pad1) -> COLUMN4
- D80 pad 2: COLUMN4 -> Net-(D80-Pad2)
- D81 pad 1: Net-(D81-Pad1) -> COLUMN4
- D81 pad 2: COLUMN4 -> Net-(D81-Pad2)
- D82 pad 1: Net-(D82-Pad1) -> COLUMN4
- D82 pad 2: COLUMN4 -> Net-(D82-Pad2)
- D83 pad 1: Net-(D83-Pad1) -> COLUMN3
- D83 pad 2: COLUMN3 -> Net-(D83-Pad2)
- D84 pad 1: Net-(D84-Pad1) -> COLUMN3
- D84 pad 2: COLUMN3 -> Net-(D84-Pad2)
- D85 pad 1: Net-(D85-Pad1) -> COLUMN3
- D85 pad 2: COLUMN3 -> Net-(D85-Pad2)
- D86 pad 1: Net-(D86-Pad1) -> COLUMN3
- D86 pad 2: COLUMN3 -> Net-(D86-Pad2)
- D87 pad 1: Net-(D87-Pad1) -> COLUMN3
- D87 pad 2: COLUMN3 -> Net-(D87-Pad2)
- D88 pad 1: Net-(D88-Pad1) -> COLUMN3
- D88 pad 2: COLUMN3 -> Net-(D88-Pad2)
- D89 pad 1: Net-(D89-Pad1) -> COLUMN3
- D89 pad 2: COLUMN3 -> Net-(D89-Pad2)
- D9 pad 1: Net-(D9-Pad1) -> COLUMN10
- D9 pad 2: COLUMN10 -> Net-(D9-Pad2)
- D90 pad 1: Net-(D90-Pad1) -> COLUMN3
- D90 pad 2: COLUMN3 -> Net-(D90-Pad2)
- D91 pad 1: Net-(D91-Pad1) -> COLUMN3
- D91 pad 2: COLUMN3 -> Net-(D91-Pad2)
- D92 pad 1: Net-(D92-Pad1) -> COLUMN3
- D92 pad 2: COLUMN3 -> Net-(D92-Pad2)
- D93 pad 1: Net-(D93-Pad1) -> COLUMN3
- D93 pad 2: COLUMN3 -> Net-(D93-Pad2)
- D94 pad 1: Net-(D94-Pad1) -> COLUMN2
- D94 pad 2: COLUMN2 -> Net-(D94-Pad2)
- D95 pad 1: Net-(D95-Pad1) -> COLUMN2
- D95 pad 2: COLUMN2 -> Net-(D95-Pad2)
- D96 pad 1: Net-(D96-Pad1) -> COLUMN2
- D96 pad 2: COLUMN2 -> Net-(D96-Pad2)
- D97 pad 1: Net-(D97-Pad1) -> COLUMN2
- D97 pad 2: COLUMN2 -> Net-(D97-Pad2)
- D98 pad 1: Net-(D98-Pad1) -> COLUMN2
- D98 pad 2: COLUMN2 -> Net-(D98-Pad2)
- D99 pad 1: Net-(D99-Pad1) -> COLUMN2
- D99 pad 2: COLUMN2 -> Net-(D99-Pad2)
- sw1 pad 2: Net-(D1-Pad1) -> Net-(D1-Pad2)
- sw10 pad 2: Net-(D10-Pad1) -> Net-(D10-Pad2)
- sw100 pad 2: Net-(D100-Pad1) -> Net-(D100-Pad2)
- sw101 pad 2: Net-(D101-Pad1) -> Net-(D101-Pad2)
- sw102 pad 2: Net-(D102-Pad1) -> Net-(D102-Pad2)
- sw103 pad 2: Net-(D103-Pad1) -> Net-(D103-Pad2)
- sw104 pad 2: Net-(D104-Pad1) -> Net-(D104-Pad2)
- sw105 pad 2: Net-(D105-Pad1) -> Net-(D105-Pad2)
- sw106 pad 2: Net-(D106-Pad1) -> Net-(D106-Pad2)
- sw107 pad 2: Net-(D107-Pad1) -> Net-(D107-Pad2)
- sw108 pad 2: Net-(D108-Pad1) -> Net-(D108-Pad2)
- sw109 pad 2: Net-(D109-Pad1) -> Net-(D109-Pad2)
- sw11 pad 2: Net-(D11-Pad1) -> Net-(D11-Pad2)
- sw110 pad 2: Net-(D110-Pad1) -> Net-(D110-Pad2)
- sw111 pad 2: Net-(D111-Pad1) -> Net-(D111-Pad2)
- sw112 pad 2: Net-(D112-Pad1) -> Net-(D112-Pad2)
- sw113 pad 2: Net-(D113-Pad1) -> Net-(D113-Pad2)
- sw114 pad 2: Net-(D114-Pad1) -> Net-(D114-Pad2)
- sw115 pad 2: Net-(D115-Pad1) -> Net-(D115-Pad2)
- sw12 pad 2: Net-(D12-Pad1) -> Net-(D12-Pad2)
- sw13 pad 2: Net-(D13-Pad1) -> Net-(D13-Pad2)
- sw14 pad 2: Net-(D14-Pad1) -> Net-(D14-Pad2)
- sw15 pad 2: Net-(D15-Pad1) -> Net-(D15-Pad2)
- sw16 pad 2: Net-(D16-Pad1) -> Net-(D16-Pad2)
- sw17 pad 2: Net-(D17-Pad1) -> Net-(D17-Pad2)
- sw18 pad 2: Net-(D18-Pad1) -> Net-(D18-Pad2)
- sw19 pad 2: Net-(D19-Pad1) -> Net-(D19-Pad2)
- sw2 pad 2: Net-(D2-Pad1) -> Net-(D2-Pad2)
- sw20 pad 2: Net-(D20-Pad1) -> Net-(D20-Pad2)
- sw21 pad 2: Net-(D21-Pad1) -> Net-(D21-Pad2)
- sw22 pad 2: Net-(D22-Pad1) -> Net-(D22-Pad2)
- sw23 pad 2: Net-(D23-Pad1) -> Net-(D23-Pad2)
- sw24 pad 2: Net-(D24-Pad1) -> Net-(D24-Pad2)
- sw25 pad 2: Net-(D25-Pad1) -> Net-(D25-Pad2)
- sw26 pad 2: Net-(D26-Pad1) -> Net-(D26-Pad2)
- sw27 pad 2: Net-(D27-Pad1) -> Net-(D27-Pad2)
- sw28 pad 2: Net-(D28-Pad1) -> Net-(D28-Pad2)
- sw29 pad 2: Net-(D29-Pad1) -> Net-(D29-Pad2)
- sw3 pad 2: Net-(D3-Pad1) -> Net-(D3-Pad2)
- sw30 pad 2: Net-(D30-Pad1) -> Net-(D30-Pad2)
- sw31 pad 2: Net-(D31-Pad1) -> Net-(D31-Pad2)
- sw32 pad 2: Net-(D32-Pad1) -> Net-(D32-Pad2)
- sw33 pad 2: Net-(D33-Pad1) -> Net-(D33-Pad2)
- sw34 pad 2: Net-(D34-Pad1) -> Net-(D34-Pad2)
- sw35 pad 2: Net-(D35-Pad1) -> Net-(D35-Pad2)
- sw36 pad 2: Net-(D36-Pad1) -> Net-(D36-Pad2)
- sw37 pad 2: Net-(D37-Pad1) -> Net-(D37-Pad2)
- sw38 pad 2: Net-(D38-Pad1) -> Net-(D38-Pad2)
- sw39 pad 2: Net-(D39-Pad1) -> Net-(D39-Pad2)
- sw4 pad 2: Net-(D4-Pad1) -> Net-(D4-Pad2)
- sw40 pad 2: Net-(D40-Pad1) -> Net-(D40-Pad2)
- sw41 pad 2: Net-(D41-Pad1) -> Net-(D41-Pad2)
- sw42 pad 2: Net-(D42-Pad1) -> Net-(D42-Pad2)
- sw43 pad 2: Net-(D43-Pad1) -> Net-(D43-Pad2)
- sw44 pad 2: Net-(D44-Pad1) -> Net-(D44-Pad2)
- sw45 pad 2: Net-(D45-Pad1) -> Net-(D45-Pad2)
- sw46 pad 2: Net-(D46-Pad1) -> Net-(D46-Pad2)
- sw47 pad 2: Net-(D47-Pad1) -> Net-(D47-Pad2)
- sw48 pad 2: Net-(D48-Pad1) -> Net-(D48-Pad2)
- sw49 pad 2: Net-(D49-Pad1) -> Net-(D49-Pad2)
- sw5 pad 2: Net-(D5-Pad1) -> Net-(D5-Pad2)
- sw50 pad 2: Net-(D50-Pad1) -> Net-(D50-Pad2)
- sw51 pad 2: Net-(D51-Pad1) -> Net-(D51-Pad2)
- sw52 pad 2: Net-(D52-Pad1) -> Net-(D52-Pad2)
- sw53 pad 2: Net-(D53-Pad1) -> Net-(D53-Pad2)
- sw54 pad 2: Net-(D54-Pad1) -> Net-(D54-Pad2)
- sw55 pad 2: Net-(D55-Pad1) -> Net-(D55-Pad2)
- sw56 pad 2: Net-(D56-Pad1) -> Net-(D56-Pad2)
- sw57 pad 2: Net-(D57-Pad1) -> Net-(D57-Pad2)
- sw58 pad 2: Net-(D58-Pad1) -> Net-(D58-Pad2)
- sw59 pad 2: Net-(D59-Pad1) -> Net-(D59-Pad2)
- sw6 pad 2: Net-(D6-Pad1) -> Net-(D6-Pad2)
- sw60 pad 2: Net-(D60-Pad1) -> Net-(D60-Pad2)
- sw61 pad 2: Net-(D61-Pad1) -> Net-(D61-Pad2)
- sw62 pad 2: Net-(D62-Pad1) -> Net-(D62-Pad2)
- sw63 pad 2: Net-(D63-Pad1) -> Net-(D63-Pad2)
- sw64 pad 2: Net-(D64-Pad1) -> Net-(D64-Pad2)
- sw65 pad 2: Net-(D65-Pad1) -> Net-(D65-Pad2)
- sw66 pad 2: Net-(D66-Pad1) -> Net-(D66-Pad2)
- sw67 pad 2: Net-(D67-Pad1) -> Net-(D67-Pad2)
- sw68 pad 2: Net-(D68-Pad1) -> Net-(D68-Pad2)
- sw69 pad 2: Net-(D69-Pad1) -> Net-(D69-Pad2)
- sw7 pad 2: Net-(D7-Pad1) -> Net-(D7-Pad2)
- sw70 pad 2: Net-(D70-Pad1) -> Net-(D70-Pad2)
- sw71 pad 2: Net-(D71-Pad1) -> Net-(D71-Pad2)
- sw72 pad 2: Net-(D72-Pad1) -> Net-(D72-Pad2)
- sw73 pad 2: Net-(D73-Pad1) -> Net-(D73-Pad2)
- sw74 pad 2: Net-(D74-Pad1) -> Net-(D74-Pad2)
- sw75 pad 2: Net-(D75-Pad1) -> Net-(D75-Pad2)
- sw76 pad 2: Net-(D76-Pad1) -> Net-(D76-Pad2)
- sw77 pad 2: Net-(D77-Pad1) -> Net-(D77-Pad2)
- sw78 pad 2: Net-(D78-Pad1) -> Net-(D78-Pad2)
- sw79 pad 2: Net-(D79-Pad1) -> Net-(D79-Pad2)
- sw8 pad 2: Net-(D8-Pad1) -> Net-(D8-Pad2)
- sw80 pad 2: Net-(D80-Pad1) -> Net-(D80-Pad2)
- sw81 pad 2: Net-(D81-Pad1) -> Net-(D81-Pad2)
- sw82 pad 2: Net-(D82-Pad1) -> Net-(D82-Pad2)
- sw83 pad 2: Net-(D83-Pad1) -> Net-(D83-Pad2)
- sw84 pad 2: Net-(D84-Pad1) -> Net-(D84-Pad2)
- sw85 pad 2: Net-(D85-Pad1) -> Net-(D85-Pad2)
- sw86 pad 2: Net-(D86-Pad1) -> Net-(D86-Pad2)
- sw87 pad 2: Net-(D87-Pad1) -> Net-(D87-Pad2)
- sw88 pad 2: Net-(D88-Pad1) -> Net-(D88-Pad2)
- sw89 pad 2: Net-(D89-Pad1) -> Net-(D89-Pad2)
- sw9 pad 2: Net-(D9-Pad1) -> Net-(D9-Pad2)
- sw90 pad 2: Net-(D90-Pad1) -> Net-(D90-Pad2)
- sw91 pad 2: Net-(D91-Pad1) -> Net-(D91-Pad2)
- sw92 pad 2: Net-(D92-Pad1) -> Net-(D92-Pad2)
- sw93 pad 2: Net-(D93-Pad1) -> Net-(D93-Pad2)
- sw94 pad 2: Net-(D94-Pad1) -> Net-(D94-Pad2)
- sw95 pad 2: Net-(D95-Pad1) -> Net-(D95-Pad2)
- sw96 pad 2: Net-(D96-Pad1) -> Net-(D96-Pad2)
- sw97 pad 2: Net-(D97-Pad1) -> Net-(D97-Pad2)
- sw98 pad 2: Net-(D98-Pad1) -> Net-(D98-Pad2)
- sw99 pad 2: Net-(D99-Pad1) -> Net-(D99-Pad2)
Routing:
- net COLUMN10: track 349.1 -> 330.4 mm
- net Net-(D75-Pad1): track 9.14 -> 0.00 mm
- net Net-(D51-Pad2): track 0.00 -> 8.96 mm
- net Net-(D75-Pad2): track 0.00 -> 8.85 mm
- net Net-(D52-Pad1): track 8.67 -> 0.00 mm
- net Net-(D44-Pad1): track 8.67 -> 0.00 mm
- net Net-(D112-Pad1): track 8.67 -> 0.00 mm
- net Net-(D111-Pad1): track 8.67 -> 0.00 mm
- net Net-(D107-Pad1): track 8.67 -> 0.00 mm
- net Net-(D100-Pad1): track 8.67 -> 0.00 mm
- net Net-(D95-Pad1): track 8.67 -> 0.00 mm
- net Net-(D73-Pad1): track 8.67 -> 0.00 mm
- net Net-(D106-Pad1): track 8.67 -> 0.00 mm
- net Net-(D78-Pad1): track 8.67 -> 0.00 mm
- net Net-(D70-Pad1): track 8.67 -> 0.00 mm
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