File: kicad/_autosave-kicad.kicad_pcb (KiCad board)
At the start: 2 copper layers, 198 parts, among them J1 USB_B_Micro, J2 SWD, J3 pwr_led+, J4 pwr_led-, J5 caps_led+, J6 caps_led-, U1 AMS1117-3.3, Y1 16MGz, sw1 Esc, sw10 Z, sw11 LCtrl, sw12 LSys, sw13 F2, sw14 F3, sw15 2, sw16 3, sw17 W, sw18 E, sw19 S, sw2 F1, sw20 D, sw21 X, sw22 C, sw23 LAlt, sw24 THome, sw25 F4, sw26 F5, sw27 4, sw28 5, sw29 R, sw3 Tilda, sw30 T, sw31 F, sw32 G, sw33 V, sw34 B, sw35 LSpace, sw36 TLeft, sw37 F6, sw38 F7, sw39 6, sw4 1, sw40 7, sw41 Y, sw42 U, sw43 H, sw44 J, sw45 N, sw46 M, sw47 TUp, sw48 TDown, sw49 F8, sw5 Tab, sw50 F9, sw51 8, sw52 9, sw53 I, sw54 O, sw55 K, sw56 L, sw57 Comma, sw58 Period, sw59 RSpace, sw6 Q, sw60 TRight, sw61 F10, sw62 F11, sw63 0, sw64 Minus, sw65 P, sw66 LBrack, sw67 Semi, sw68 Quote, sw69 FSlash, sw7 CAPS, sw70 RShift, sw71 RAlt, sw72 TEnd, sw73 F12, sw74 PrtSc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

Commit message: wip
Connections:
- D1 pad 1: COLUMN10 -> COLUMN1
- D10 pad 1: COLUMN10 -> Net-(D10-K)
- D11 pad 1: COLUMN10 -> COLUMN1
- D12 pad 1: COLUMN10 -> Net-(D10-K)
- D13 pad 1: COLUMN9 -> COLUMN4
- D14 pad 1: COLUMN9 -> COLUMN5
- D15 pad 1: COLUMN9 -> COLUMN3
- D16 pad 1: COLUMN9 -> COLUMN4
- D17 pad 1: COLUMN9 -> COLUMN3
- D18 pad 1: COLUMN9 -> COLUMN4
- D19 pad 1: COLUMN9 -> COLUMN3
- D2 pad 1: COLUMN10 -> COLUMN3
- D20 pad 1: COLUMN9 -> COLUMN4
- D21 pad 1: COLUMN9 -> COLUMN3
- D22 pad 1: COLUMN9 -> COLUMN4
- D23 pad 1: COLUMN9 -> COLUMN3
- D24 pad 1: COLUMN9 -> COLUMN4
- D25 pad 1: COLUMN8 -> COLUMN6
- D26 pad 1: COLUMN8 -> COLUMN7
- D27 pad 1: COLUMN8 -> COLUMN5
- D28 pad 1: COLUMN8 -> COLUMN6
- D29 pad 1: COLUMN8 -> COLUMN5
- D3 pad 1: COLUMN10 -> COLUMN1
- D30 pad 1: COLUMN8 -> COLUMN6
- D31 pad 1: COLUMN8 -> COLUMN5
- D32 pad 1: COLUMN8 -> COLUMN6
- D33 pad 1: COLUMN8 -> COLUMN5
- D34 pad 1: COLUMN8 -> COLUMN6
- D35 pad 1: COLUMN8 -> COLUMN4
- D36 pad 1: COLUMN8 -> COLUMN5
- D37 pad 1: COLUMN7 -> COLUMN8
- D38 pad 1: COLUMN7 -> COLUMN9
- D4 pad 1: COLUMN10 -> Net-(D10-K)
- D40 pad 1: COLUMN7 -> COLUMN8
- D42 pad 1: COLUMN7 -> COLUMN8
- D44 pad 1: COLUMN7 -> COLUMN8
- D46 pad 1: COLUMN7 -> COLUMN8
- D47 pad 1: COLUMN7 -> COLUMN6
- D48 pad 1: COLUMN7 -> COLUMN6
- D49 pad 1: COLUMN6 -> COLUMN10
- D5 pad 1: COLUMN10 -> COLUMN1
- D50 pad 1: COLUMN6 -> COLUMN11
- D51 pad 1: COLUMN6 -> COLUMN9
- D52 pad 1: COLUMN6 -> COLUMN10
- D53 pad 1: COLUMN6 -> COLUMN9
- D54 pad 1: COLUMN6 -> COLUMN10
- D55 pad 1: COLUMN6 -> COLUMN9
- D56 pad 1: COLUMN6 -> COLUMN10
- D57 pad 1: COLUMN6 -> COLUMN9
- D58 pad 1: COLUMN6 -> COLUMN10
- D59 pad 1: COLUMN6 -> COLUMN8
- D6 pad 1: COLUMN10 -> Net-(D10-K)
- D60 pad 1: COLUMN6 -> COLUMN7
- D61 pad 1: COLUMN5 -> COLUMN12
- D62 pad 1: COLUMN5 -> COLUMN13
- D63 pad 1: COLUMN5 -> COLUMN11
- D64 pad 1: COLUMN5 -> COLUMN12
- D65 pad 1: COLUMN5 -> COLUMN11
- D66 pad 1: COLUMN5 -> COLUMN12
- D67 pad 1: COLUMN5 -> COLUMN11
- D68 pad 1: COLUMN5 -> COLUMN12
- D69 pad 1: COLUMN5 -> COLUMN11
- D7 pad 1: COLUMN10 -> COLUMN1
- D70 pad 1: COLUMN5 -> COLUMN14
- D71 pad 1: COLUMN5 -> COLUMN10
- D72 pad 1: COLUMN5 -> COLUMN8
- D73 pad 1: COLUMN4 -> COLUMN14
- D74 pad 1: COLUMN4 -> COLUMN13
- D75 pad 1: COLUMN4 -> COLUMN13
- D76 pad 1: COLUMN4 -> COLUMN14
- D77 pad 1: COLUMN4 -> COLUMN13
- D78 pad 1: COLUMN4 -> COLUMN14
- D79 pad 1: COLUMN4 -> COLUMN14
- D8 pad 1: COLUMN10 -> Net-(D10-K)
- D80 pad 1: COLUMN4 -> COLUMN14
- D81 pad 1: COLUMN4 -> COLUMN11
- D82 pad 1: COLUMN4 -> COLUMN12
- D85 pad 1: COLUMN3 -> COLUMN13
- D87 pad 1: COLUMN3 -> COLUMN13
- D9 pad 1: COLUMN10 -> COLUMN1
- D96 pad 1: COLUMN2 -> COLUMN3
- D98 pad 1: COLUMN2 -> COLUMN9
- MCU1 pad 39: ROW2 -> COLUMN2
- sw10 pad 1: ROW10 -> ROW5
- sw11 pad 1: ROW11 -> ROW6
- sw12 pad 1: ROW12 -> ROW6
- sw14 pad 1: ROW2 -> ROW1
- sw15 pad 1: ROW3 -> COLUMN2
- sw16 pad 1: ROW4 -> COLUMN2
- sw17 pad 1: ROW5 -> ROW3
- sw18 pad 1: ROW6 -> ROW3
- sw19 pad 1: ROW7 -> ROW4
- sw2 pad 1: ROW2 -> ROW1
- sw20 pad 1: ROW8 -> ROW4
- sw21 pad 1: ROW9 -> ROW5
- sw22 pad 1: ROW10 -> ROW5
- sw23 pad 1: ROW11 -> ROW6
- sw24 pad 1: ROW12 -> ROW7
- sw26 pad 1: ROW2 -> ROW1
- sw27 pad 1: ROW3 -> COLUMN2
- sw28 pad 1: ROW4 -> COLUMN2
- sw29 pad 1: ROW5 -> ROW3
- sw3 pad 1: ROW3 -> COLUMN2
- sw30 pad 1: ROW6 -> ROW3
- sw31 pad 1: ROW7 -> ROW4
- sw32 pad 1: ROW8 -> ROW4
- sw33 pad 1: ROW9 -> ROW5
- sw34 pad 1: ROW10 -> ROW5
- sw35 pad 1: ROW11 -> ROW6
- sw36 pad 1: ROW12 -> ROW7
- sw38 pad 1: ROW2 -> ROW1
- sw39 pad 1: ROW3 -> COLUMN2
- sw4 pad 1: ROW4 -> COLUMN2
- sw40 pad 1: ROW4 -> COLUMN2
- sw41 pad 1: ROW5 -> ROW3
- sw42 pad 1: ROW6 -> ROW3
- sw43 pad 1: ROW7 -> ROW4
- sw44 pad 1: ROW8 -> ROW4
- sw45 pad 1: ROW9 -> ROW5
- sw46 pad 1: ROW10 -> ROW5
- sw47 pad 1: ROW11 -> ROW6
- sw48 pad 1: ROW12 -> ROW7
- sw5 pad 1: ROW5 -> ROW3
- sw50 pad 1: ROW2 -> ROW1
- sw51 pad 1: ROW3 -> COLUMN2
- sw52 pad 1: ROW4 -> COLUMN2
- sw53 pad 1: ROW5 -> ROW3
- sw54 pad 1: ROW6 -> ROW3
- sw55 pad 1: ROW7 -> ROW4
- sw56 pad 1: ROW8 -> ROW4
- sw57 pad 1: ROW9 -> ROW5
- sw58 pad 1: ROW10 -> ROW5
- sw59 pad 1: ROW11 -> ROW6
- sw6 pad 1: ROW6 -> ROW3
- sw60 pad 1: ROW12 -> ROW7
- sw62 pad 1: ROW2 -> ROW1
- sw63 pad 1: ROW3 -> COLUMN2
- sw64 pad 1: ROW4 -> COLUMN2
- sw65 pad 1: ROW5 -> ROW3
- sw66 pad 1: ROW6 -> ROW3
- sw67 pad 1: ROW7 -> ROW4
- sw68 pad 1: ROW8 -> ROW4
- sw69 pad 1: ROW9 -> ROW5
- sw7 pad 1: ROW7 -> ROW4
- sw70 pad 1: ROW10 -> ROW5
- sw71 pad 1: ROW11 -> ROW6
- sw72 pad 1: ROW12 -> ROW7
- sw74 pad 1: ROW2 -> ROW6
- sw75 pad 1: ROW3 -> COLUMN2
- sw76 pad 1: ROW4 -> COLUMN2
- sw77 pad 1: ROW5 -> ROW3
- sw78 pad 1: ROW6 -> ROW3
- sw79 pad 1: ROW7 -> ROW4
- sw8 pad 1: ROW8 -> ROW4
- sw80 pad 1: ROW10 -> ROW6
- sw81 pad 1: ROW11 -> ROW6
- sw82 pad 1: ROW12 -> ROW6
- sw85 pad 1: ROW3 -> ROW5
- sw87 pad 1: ROW5 -> ROW4
- sw9 pad 1: ROW9 -> ROW5
- sw96 pad 1: ROW3 -> ROW7
- sw98 pad 1: ROW5 -> ROW7
Routing:
- net ROW1: track 19.6 -> 316.8 mm
- net ROW5: track 20.9 -> 304.4 mm
- net ROW2: track 19.6 -> 0.00 mm
- net COLUMN2: track 25.4 -> 45.0 mm
